File: PCB/Left/SofleKeyboard.kicad_pcb (KiCad board)
At the start: 2 copper layers, 217.8 x 109.2 mm, 56 parts, among them J1 Conn_01x08, J2 , SW1 1u, SW10 1u, SW11 1u, SW12 1u, SW13 1u, SW14 1u, SW15 1u, SW16 1u, SW17 1u, SW18 1u, SW19 1u, SW2 1u, SW20 1u, SW21 1u, SW22 1u, SW23 1u, SW24 1u, SW25 Rotary_Encoder_Switch, SW26 1.5u, SW27 1u, SW28 1u, SW29 1u, SW3 1u, SW30 1u, SW31 1u, SW32 1u, SW33 1u, SW34 1u, SW35 1u, SW36 1u, SW37 1u, SW38 1u, SW39 1u, SW4 1u, SW40 1u, SW41 1u, SW42 1u, SW43 1u, SW44 1u, SW45 1u, SW46 1u, SW5 1u, SW6 1u, SW7 1u, SW8 1u, SW9 1u, U4 MS88FS3

Commit message: cap nhat 16:16 08/06/2022
Parts:
- added SW48: Power Switch, Button_Switch_SMD:SW_SPDT_PCM12, B.Cu at (238.8, 30.5)
- moved U4 0.25 mm to (231.9, 42.7)
Connections:
- U4 pad 29: CHARGE_CTRL_1 -> unconnected-(U4-Pad29)
- U4 pad 30: CHARGE_CTRL_2 -> unconnected-(U4-Pad30)
- U4 pad 31: VDD -> nRF_VDD
- U4 pad 32: VDDH -> nRF_VDD
