File: PCB/nRFpill/nRFpill.kicad_pcb (KiCad board)
At the start: 2 copper layers, 52.7 x 20.8 mm, 27 parts, among them J1 USB_C_Receptacle_USB2.0, J2 , J3 , Q1 AO3407, Q2 AO3407, SW1 RST, SW2 DFU, U1 MIC5219-3.3YM5, U2 USBLC6-2SC6, U3 TP4054, U5 MS88FS3

Commit message: cap nhat luc nua dem 23:54 12/06/2022
Parts:
- added C1: 100nF, Capacitor_SMD:C_0603_1608Metric, F.Cu at (73.7, 51.9)
- added J4: , TestPoint:TestPoint_Pad_1.5x1.5mm, B.Cu at (58.4, 50.8)
- added J5: , TestPoint:TestPoint_Pad_D1.5mm, B.Cu at (61.0, 50.8)
- added R1: 2M, Resistor_SMD:R_0603_1608Metric, F.Cu at (76.3, 54.2)
- added R3: 2M, Resistor_SMD:R_0603_1608Metric, F.Cu at (74.4, 54.2)
- added R7: 10M, Resistor_SMD:R_0603_1608Metric, F.Cu at (72.9, 54.2)
- moved R9 3.15 mm to (76.3, 51.1)
- moved R10 2.84 mm to (73.7, 50.3), turned to 180 degrees
Connections:
- J2 pad 1: unconnected-(J2-Pad1) -> 1.02
- J2 pad 10: unconnected-(J2-Pad10) -> 0.17
- J2 pad 11: unconnected-(J2-Pad11) -> 0.21
- J2 pad 12: unconnected-(J2-Pad12) -> 0.23
- J2 pad 13: unconnected-(J2-Pad13) -> 0.20
- J2 pad 14: unconnected-(J2-Pad14) -> 0.22
- J2 pad 15: unconnected-(J2-Pad15) -> 0.24
- J2 pad 16: unconnected-(J2-Pad16) -> 1.00
- J2 pad 17: unconnected-(J2-Pad17) -> 0.25
- J2 pad 2: unconnected-(J2-Pad2) -> 0.12
- J2 pad 3: unconnected-(J2-Pad3) -> 0.16
- J2 pad 4: unconnected-(J2-Pad4) -> 0.14
- J2 pad 5: unconnected-(J2-Pad5) -> 0.19
- J2 pad 6: unconnected-(J2-Pad6) -> 0.13
- J2 pad 7: unconnected-(J2-Pad7) -> 0.15
- J3 pad 10: unconnected-(J3-Pad10) -> 0.07
- J3 pad 11: unconnected-(J3-Pad11) -> 0.31
- J3 pad 12: unconnected-(J3-Pad12) -> 0.30
- J3 pad 13: unconnected-(J3-Pad13) -> 0.26
- J3 pad 14: unconnected-(J3-Pad14) -> 0.05
- J3 pad 15: unconnected-(J3-Pad15) -> 0.27
- J3 pad 19: unconnected-(J3-Pad19) -> LED_1
- J3 pad 4: unconnected-(J3-Pad4) -> 1.09
- J3 pad 5: unconnected-(J3-Pad5) -> 0.28
- J3 pad 6: unconnected-(J3-Pad6) -> 0.08
- J3 pad 7: unconnected-(J3-Pad7) -> 0.11
- J3 pad 8: unconnected-(J3-Pad8) -> 1.08
- J3 pad 9: unconnected-(J3-Pad9) -> 0.06
- U5 pad 10: 0.29 -> unconnected-(U5-Pad10)
- U5 pad 2: 1.11 -> unconnected-(U5-Pad2)
- U5 pad 3: 1.12 -> unconnected-(U5-Pad3)
- U5 pad 4: 1.10 -> unconnected-(U5-Pad4)
- U5 pad 5: 1.14 -> unconnected-(U5-Pad5)
- U5 pad 53: 1.04 -> unconnected-(U5-Pad53)
- U5 pad 54: DFU -> LED_2
- U5 pad 55: LED_2 -> DFU
- U5 pad 57: 1.07 -> unconnected-(U5-Pad57)
- U5 pad 58: 1.05 -> unconnected-(U5-Pad58)
- U5 pad 59: 1.01 -> unconnected-(U5-Pad59)
- U5 pad 6: 0.03 -> unconnected-(U5-Pad6)
- U5 pad 60: 1.03 -> unconnected-(U5-Pad60)
- U5 pad 7: 1.13 -> unconnected-(U5-Pad7)
- U5 pad 8: 1.15 -> unconnected-(U5-Pad8)
- U5 pad 9: 0.02 -> unconnected-(U5-Pad9)
Routing:
- net 1.02: track 0.00 -> 50.7 mm, vias 0 -> 1
- net LED_1: track 0.00 -> 45.1 mm, vias 0 -> 2
- net 0.12: track 0.00 -> 34.2 mm, vias 0 -> 2
- net DP+: track 5.82 -> 38.5 mm
- net 0.28: track 0.00 -> 32.5 mm, vias 0 -> 1
- net DFU: track 0.00 -> 32.2 mm, vias 0 -> 2
- net LED_2: track 0.00 -> 32.0 mm, vias 0 -> 2
- net 0.19: track 0.00 -> 31.5 mm, vias 0 -> 1
- net 0.16: track 0.00 -> 30.7 mm, vias 0 -> 1
- net 0.13: track 0.00 -> 29.0 mm, vias 0 -> 1
- net 1.09: track 0.00 -> 28.9 mm, vias 0 -> 1
- net 0.14: track 0.00 -> 28.0 mm, vias 0 -> 1
- net 0.15: track 0.00 -> 27.2 mm, vias 0 -> 1
- net DP-: track 5.97 -> 30.7 mm, vias 0 -> 1
- net 0.08: track 0.00 -> 23.6 mm, vias 0 -> 1
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- added copper zone on B.Cu, net (none)
- added copper zone on F.Cu, net (none)

Commit message: cap nhat 11:55 13/06/2022
Parts:
- U1, U3: footprint Package_TO_SOT_SMD:SOT-23-5 -> Library:SOT-23-5
- U2: footprint Package_TO_SOT_SMD:SOT-23-6 -> Library:SOT-23-6
- moved R11 0.28 mm to (91.6, 47.1)
- moved R5 0.28 mm to (91.6, 54.4)
Connections:
- J2 pad 1: 1.02 -> 1.07
- U5 pad 52: 1.02 -> unconnected-(U5-Pad52)
- U5 pad 54: LED_2 -> unconnected-(U5-Pad54)
- U5 pad 55: DFU -> unconnected-(U5-Pad55)
- U5 pad 56: LED_1 -> unconnected-(U5-Pad56)
- U5 pad 57: unconnected-(U5-Pad57) -> 1.07
- U5 pad 58: unconnected-(U5-Pad58) -> LED_1
- U5 pad 59: unconnected-(U5-Pad59) -> DFU
- U5 pad 60: unconnected-(U5-Pad60) -> LED_2
Routing:
- net 1.07: track 0.00 -> 52.4 mm, vias 0 -> 1
- net 1.02: track 50.7 -> 0.00 mm, vias 1 -> 0
- net LED_2: track 32.0 -> 28.8 mm
- net DFU: track 32.2 -> 30.3 mm
- net LED_1: track 45.1 -> 45.7 mm
- net GND: track 27.9 -> 27.3 mm
Other:
- board text added: "+5V"
- board text added: "0.1"
- board text added: "000"
- board text added: "001"
- board text added: "005"
- board text added: "006"
- board text added: "007"
- board text added: "008"
- board text added: "011"
- board text added: "012"
- board text added: "013"
- board text added: "014"
- board text added: "015"
- board text added: "016"
- board text added: "017"
- board text added: "019"
- board text added: "020"
- board text added: "021"
- board text added: "022"
- board text added: "023"
- board text added: "024"
- board text added: "025"
- board text added: "026"
- board text added: "027"
- board text added: "028"
- board text added: "030"
- board text added: "031"
- board text added: "100"
- board text added: "105"
- board text added: "107"
- board text added: "108"
- board text added: "109"
- board text added: "CLK"
- board text added: "DFU"
- board text added: "DIO"
- board text added: "GND"
- board text added: "LED1"
- board text added: "LED2"
- board text added: "RST"
- board text added: "VBAT"
- board text added: "nRF Pill"
- board text removed: "5V"
- board text removed: "G"
