File: PCB/nRFpill/nRFpill.kicad_sch (KiCad schematic)
At the start: 33 parts, among them J1 USB_C_Receptacle_USB2.0, J2 , J3 , Q1 AO3407, Q2 AO3407, SW1 RST, SW2 DFU, U1 MIC5219-3.3YM5, U2 USBLC6-2SC6, U3 TP4054, U4 Blackpill-F4x1, U5 MS88FS3

Commit message: cap nhat luc nua dem 23:54 12/06/2022
Parts:
- removed SWD1: SWD-STM32-4Pin, kien242:SWD-4Pin, symbol keni242:SWD-STM32-4Pin
- removed U4: Blackpill-F4x1, symbol kien242:Blackpill-F4x1
- added J4: (no value), TestPoint:TestPoint_Pad_1.5x1.5mm, symbol Connector_Generic:Conn_01x01
- added J5: (no value), TestPoint:TestPoint_Pad_D1.5mm, symbol Connector_Generic:Conn_01x01
Connections:
- net 0.02: no longer U5.9 (0.02/AIN0)
- net 0.03: no longer U5.6 (0.03/AIN1)
- net 0.05: now also J3.14 (Pin_14)
- net 0.06: now also J3.9 (Pin_9)
- net 0.07: now also J3.10 (Pin_10)
- net 0.08: now also J3.6 (Pin_6)
- net 0.11: now also J3.7 (Pin_7)
- net 0.12: now also J2.2 (Pin_2)
- net 0.13: now also J2.6 (Pin_6)
- net 0.14: now also J2.4 (Pin_4)
- net 0.15: now also J2.7 (Pin_7)
- net 0.16: now also J2.3 (Pin_3)
- net 0.17: now also J2.10 (Pin_10)
- net 0.19: now also J2.5 (Pin_5)
- net 0.20: now also J2.13 (Pin_13)
- net 0.21: now also J2.11 (Pin_11)
- net 0.22: now also J2.14 (Pin_14)
- net 0.23: now also J2.12 (Pin_12)
- net 0.24: now also J2.15 (Pin_15)
- net 0.25: now also J2.17 (Pin_17)
- net 0.26: now also J3.13 (Pin_13)
- net 0.27: now also J3.15 (Pin_15)
- net 0.28: now also J3.5 (Pin_5)
- net 0.29: no longer U5.10 (0.29/AIN5)
- net 0.30: now also J3.12 (Pin_12)
- net 0.31: now also J3.11 (Pin_11)
- net 1.00: now also J2.16 (Pin_16)
- net 1.01: no longer U5.59 (1.01)
- net 1.02: now also J2.1 (Pin_1)
- net 1.03: no longer U5.60 (1.03)
- net 1.05: no longer U5.58 (1.05)
- net 1.07: no longer U5.57 (1.07)
- net 1.08: now also J3.8 (Pin_8)
- net 1.09: now also J3.4 (Pin_4)
- net 1.10: no longer U5.4 (1.10)
- net 1.11: no longer U5.2 (1.11)
- net 1.12: no longer U5.3 (1.12)
- net 1.13: no longer U5.7 (1.13)
- net 1.14: no longer U5.5 (1.14)
- net 1.15: no longer U5.8 (1.15)
- net DFU: now also U5.55 (0.09); no longer U5.54 (1.06)
- net LED_1: now also J3.19 (Pin_19)
- net LED_2: now also U5.54 (1.06); no longer U5.55 (0.09)
- net SWCLK: now also J4.1 (Pin_1)
- net SWDIO: now also J5.1 (Pin_1)
- net 1.04: no longer names the net of U5.53 (1.04)
Other:
- moved on the sheet: J3

Commit message: cap nhat 11:55 13/06/2022
Parts:
- U1, U3: footprint Package_TO_SOT_SMD:SOT-23-5 -> Library:SOT-23-5
- U2: footprint Package_TO_SOT_SMD:SOT-23-6 -> Library:SOT-23-6
Connections:
- net 1.07: now also J2.1 (Pin_1), U5.57 (1.07)
- net DFU: now also U5.59 (1.01); no longer U5.55 (0.09)
- net LED_1: now also U5.58 (1.05); no longer U5.56 (0.10)
- net LED_2: now also U5.60 (1.03); no longer U5.54 (1.06)
- net 1.02: no longer names the net of U5.52 (1.02)
- net 1.02: no longer J2.1 (Pin_1)
Changed lines of the file:
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@@
-    )
-  )
-  (global_label "1.05" (shape input) (at 160.02 80.645 0) (fields_autoplaced)
-    (effects (font (size 1.27 1.27)) (justify left))
-    (property "Intersheet References" "${INTERSHEET_REFS}" (id 0) (at 166.6664 80.5656 0)
-      (effects (font (size 1.27 1.27)) (justify left) hide)
     )
   )
@@
     (property "Intersheet References" "${INTERSHEET_REFS}" (id 0) (at 265.7686 125.6506 0)
       (effects (font (size 1.27 1.27)) (justify right) hide)
-    )
-  )
-  (global_label "1.01" (shape input) (at 160.02 83.185 0) (fields_autoplaced)
-    (effects (font (size 1.27 1.27)) (justify left))
-    (property "Intersheet References" "${INTERSHEET_REFS}" (id 0) (at 166.6664 83.1056 0)
-      (effects (font (size 1.27 1.27)) (justify left) hide)
     )
   )
@@
     )
   )
+  (global_label "DFU" (shape input) (at 158.75 83.185 0) (fields_autoplaced)
+    (effects (font (size 1.27 1.27)) (justify left))
+    (property "Intersheet References" "${INTERSHEET_REFS}" (id 0) (at 164.8521 83.2644 0)
+      (effects (font (size 1.27 1.27)) (justify right) hide)
+    )
+  )
   (global_label "0.06" (shape input) (at 115.57 141.605 270) (fields_autoplaced)
     (effects (font (size 1.27 1.27)) (justify right))
@@
     )
   )
-  (global_label "LED_2" (shape input) (at 143.51 70.485 90) (fields_autoplaced)
-    (effects (font (size 1.27 1.27)) (justify left))
-    (property "Intersheet References" "${INTERSHEET_REFS}" (id 0) (at 143.5894 62.4476 90)
-      (effects (font (size 1.27 1.27)) (justify right) hide)
-    )
-  )
   (global_label "0.24" (shape input) (at 158.75 103.505 0) (fields_autoplaced)
     (effects (font (size 1.27 1.27)) (justify left))
@@
     )
   )
-  (global_label "1.02" (shape input) (at 253.365 90.17 0) (fields_autoplaced)
+  (global_label "1.07" (shape input) (at 253.365 90.17 0) (fields_autoplaced)
     (effects (font (size 1.27 1.27)) (justify left))
     (property "Intersheet References" "${INTERSHEET_REFS}" (id 0) (at 260.0114 90.0906 0)
@@
     )
   )
-  (global_label "DFU" (shape input) (at 140.97 70.485 90) (fields_autoplaced)
-    (effects (font (size 1.27 1.27)) (justify left))
-    (property "Intersheet References" "${INTERSHEET_REFS}" (id 0) (at 141.0494 64.3829 90)
-      (effects (font (size 1.27 1.27)) (justify right) hide)
-    )
-  )
   (global_label "0.20" (shape input) (at 158.75 108.585 0) (fields_autoplaced)
     (effects (font (size 1.27 1.27)) (justify left))
@@
     )
   )
+  (global_label "LED_2" (shape input) (at 158.75 85.725 0) (fields_autoplaced)
+    (effects (font (size 1.27 1.27)) (justify left))
+    (property "Intersheet References" "${INTERSHEET_REFS}" (id 0) (at 166.7874 85.8044 0)
+      (effects (font (size 1.27 1.27)) (justify right) hide)
+    )
+  )
   (global_label "0.14" (shape input) (at 140.97 141.605 270) (fields_autoplaced)
     (effects (font (size 1.27 1.27)) (justify right))
@@
     )
   )
-  (global_label "1.02" (shape input) (at 148.59 70.485 90) (fields_autoplaced)
-    (effects (font (size 1.27 1.27)) (justify left))
-    (property "Intersheet References" "${INTERSHEET_REFS}" (id 0) (at 148.5106 63.8386 90)
+  (global_label "1.07" (shape input) (at 158.75 78.105 0) (fields_autoplaced)
+    (effects (font (size 1.27 1.27)) (justify left))
+    (property "Intersheet References" "${INTERSHEET_REFS}" (id 0) (at 165.3964 78.0256 0)
       (effects (font (size 1.27 1.27)) (justify left) hide)
     )
@@
     )
   )
-  (global_label "LED_1" (shape input) (at 138.43 70.485 90) (fields_autoplaced)
-    (effects (font (size 1.27 1.27)) (justify left))
-    (property "Intersheet References" "${INTERSHEET_REFS}" (id 0) (at 138.5094 62.4476 90)
-      (effects (font (size 1.27 1.27)) (justify left) hide)
-    )
-  )
   (global_label "0.05" (shape input) (at 272.415 123.19 180) (fields_autoplaced)
     (effects (font (size 1.27 1.27)) (justify right))
@@
     (effects (font (size 1.27 1.27)) (justify left))
     (property "Intersheet References" "${INTERSHEET_REFS}" (id 0) (at 163.8658 126.4444 0)
+      (effects (font (size 1.27 1.27)) (justify left) hide)
+    )
+  )
+  (global_label "LED_1" (shape input) (at 158.75 80.645 0) (fields_autoplaced)
+    (effects (font (size 1.27 1.27)) (justify left))
+    (property "Intersheet References" "${INTERSHEET_REFS}" (id 0) (at 166.7874 80.7244 0)
       (effects (font (size 1.27 1.27)) (justify left) hide)
     )
@@
     )
   )
-  (global_label "1.03" (shape input) (at 160.02 85.725 0) (fields_autoplaced)
-    (effects (font (size 1.27 1.27)) (justify left))
-    (property "Intersheet References" "${INTERSHEET_REFS}" (id 0) (at 166.6664 85.6456 0)
-      (effects (font (size 1.27 1.27)) (justify left) hide)
-    )
-  )
   (global_label "0.12" (shape input) (at 253.365 92.71 0) (fields_autoplaced)
     (effects (font (size 1.27 1.27)) (justify left))
@@
     (property "Intersheet References" "${INTERSHEET_REFS}" (id 0) (at 118.0306 148.2514 90)
       (effects (font (size 1.27 1.27)) (justify right) hide)
-    )
-  )
-  (global_label "1.07" (shape input) (at 160.02 78.105 0) (fields_autoplaced)
-    (effects (font (size 1.27 1.27)) (justify left))
-    (property "Intersheet References" "${INTERSHEET_REFS}" (id 0) (at 166.6664 78.0256 0)
-      (effects (font (size 1.27 1.27)) (justify left) hide)
     )
   )
@@
     (property "Reference" "U3" (id 0) (at 42.545 170.815 0))
     (property "Value" "TP4054" (id 1) (at 42.545 173.355 0))
-    (property "Footprint" "Package_TO_SOT_SMD:SOT-23-5" (id 2) (at 41.275 188.595 0)
+    (property "Footprint" "Library:SOT-23-5" (id 2) (at 41.275 188.595 0)
       (effects (font (size 1.27 1.27) italic) (justify left) hide)
     )
@@
     (property "Reference" "U1" (id 0) (at 126.365 34.925 0))
     (property "Value" "MIC5219-3.3YM5" (id 1) (at 126.365 37.465 0))
-    (property "Footprint" "Package_TO_SOT_SMD:SOT-23-5" (id 2) (at 126.365 36.195 0)
+    (property "Footprint" "Library:SOT-23-5" (id 2) (at 126.365 36.195 0)
       (effects (font (size 1.27 1.27)) hide)
     )
@@
     (property "Reference" "U2" (id 0) (at 45.72 95.25 0))
     (property "Value" "USBLC6-2SC6" (id 1) (at 31.75 95.25 0))
-    (property "Footprint" "Package_TO_SOT_SMD:SOT-23-6" (id 2) (at 39.37 116.84 0)
+    (property "Footprint" "Library:SOT-23-6" (id 2) (at 39.37 116.84 0)
       (effects (font (size 1.27 1.27)) hide)
     )
@@
     )
     (path "/6fc07099-549a-4dc5-8c80-3ec767b4b363"
-      (reference "U1") (unit 1) (value "MIC5219-3.3YM5") (footprint "Package_TO_SOT_SMD:SOT-23-5")
+      (reference "U1") (unit 1) (value "MIC5219-3.3YM5") (footprint "Library:SOT-23-5")
     )
     (path "/dc7fe6ab-e2e1-48c0-b2af-0f1c6ebb04ac"
-      (reference "U2") (unit 1) (value "USBLC6-2SC6") (footprint "Package_TO_SOT_SMD:SOT-23-6")
+      (reference "U2") (unit 1) (value "USBLC6-2SC6") (footprint "Library:SOT-23-6")
     )
     (path "/6167ac01-a97a-4a6f-b811-bc0a02b4630c"
-      (reference "U3") (unit 1) (value "TP4054") (footprint "Package_TO_SOT_SMD:SOT-23-5")
+      (reference "U3") (unit 1) (value "TP4054") (footprint "Library:SOT-23-5")
     )
     (path "/5d9bd90f-7da9-498d-a850-139e5487556e"

Commit message: update file
Parts:
- C1: value 100nF -> 10nF
- C5: value 0.1uF -> 100nF
- R10: value RPROG -> 2k
- R6: value 2M -> 100K
Changed lines of the file:
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@@
   (symbol (lib_id "Device:C") (at 205.74 111.76 0) (unit 1)
     (in_bom yes) (on_board yes) (fields_autoplaced)
-    (property "Reference" "C5" (id 0) (at 208.915 110.4899 0)
-      (effects (font (size 1.27 1.27)) (justify left))
-    )
-    (property "Value" "0.1uF" (id 1) (at 208.915 113.0299 0)
+    (property "Reference" "C5" (id 0) (at 209.55 110.4899 0)
+      (effects (font (size 1.27 1.27)) (justify left))
+    )
+    (property "Value" "100nF" (id 1) (at 209.55 113.0299 0)
       (effects (font (size 1.27 1.27)) (justify left))
     )
@@
     (in_bom yes) (on_board yes)
     (property "Reference" "R10" (id 0) (at 56.515 179.5272 90))
-    (property "Value" "RPROG" (id 1) (at 56.515 181.8386 90))
+    (property "Value" "2k" (id 1) (at 56.515 181.8386 90))
     (property "Footprint" "Resistor_SMD:R_0603_1608Metric" (id 2) (at 56.515 183.007 90)
       (effects (font (size 1.27 1.27)) hide)
@@
   (symbol (lib_id "Device:C_Small") (at 189.865 40.64 0) (unit 1)
     (in_bom yes) (on_board yes) (fields_autoplaced)
-    (property "Reference" "C1" (id 0) (at 193.04 39.3699 0)
-      (effects (font (size 1.27 1.27)) (justify left))
-    )
-    (property "Value" "100nF" (id 1) (at 193.04 41.9099 0)
+    (property "Reference" "C1" (id 0) (at 193.04 39.3762 0)
+      (effects (font (size 1.27 1.27)) (justify left))
+    )
+    (property "Value" "10nF" (id 1) (at 193.04 41.9162 0)
       (effects (font (size 1.27 1.27)) (justify left))
     )
@@
       (effects (font (size 1.27 1.27)) (justify left))
     )
-    (property "Value" "2M" (id 1) (at 219.202 39.878 0)
+    (property "Value" "100K" (id 1) (at 219.202 39.878 0)
       (effects (font (size 1.27 1.27)) (justify left))
     )
@@
     )
     (path "/e0ff723e-9da4-419a-9b7c-537137a1c661"
-      (reference "C1") (unit 1) (value "100nF") (footprint "Capacitor_SMD:C_0603_1608Metric")
+      (reference "C1") (unit 1) (value "10nF") (footprint "Capacitor_SMD:C_0603_1608Metric")
     )
     (path "/f420da17-70b9-4289-9973-71af4d270f42"
@@
     )
     (path "/b103f2ec-3c6b-4830-96f7-70d27dea761e"
-      (reference "C5") (unit 1) (value "0.1uF") (footprint "Capacitor_SMD:C_0603_1608Metric")
+      (reference "C5") (unit 1) (value "100nF") (footprint "Capacitor_SMD:C_0603_1608Metric")
     )
     (path "/3525d7fb-9fbb-407a-b98f-dbe710a5769f"
@@
     )
     (path "/ec41bd13-d169-4b04-82e8-82bf8614a606"
-      (reference "R6") (unit 1) (value "2M") (footprint "Resistor_SMD:R_0603_1608Metric")
+      (reference "R6") (unit 1) (value "100K") (footprint "Resistor_SMD:R_0603_1608Metric")
     )
     (path "/c6be61ba-466b-4919-aa01-8bb9fa803922"
@@
     )
     (path "/dd10163f-a041-4080-beea-991cfe918582"
-      (reference "R10") (unit 1) (value "RPROG") (footprint "Resistor_SMD:R_0603_1608Metric")
+      (reference "R10") (unit 1) (value "2k") (footprint "Resistor_SMD:R_0603_1608Metric")
     )
     (path "/32eae5dc-f362-4450-8ba9-22274608b5ec"

Commit message: cap nhat
Parts:
- removed D4: BLUE, LED_SMD:LED_0603_1608Metric, symbol Device:LED
- removed R11: 1K, Resistor_SMD:R_0603_1608Metric, symbol Device:R_Small
- U: renamed from R2; value 5.1k -> (none); footprint Resistor_SMD:R_0603_1608Metric -> (none)
- U: renamed from J5; value (none) -> (none); footprint TestPoint:TestPoint_Pad_D1.5mm -> (none)
- U: renamed from R5; value 1K -> (none); footprint Resistor_SMD:R_0603_1608Metric -> (none)
- U: renamed from C4; value 10uF -> (none); footprint Capacitor_SMD:C_0603_1608Metric -> (none)
- U: renamed from D1; value BLUE -> (none); footprint LED_SMD:LED_0603_1608Metric -> (none)
- U: renamed from Q1; value AO3407 -> (none); footprint Package_TO_SOT_SMD:SOT-23 -> (none)
- U: renamed from J3; value (none) -> (none); footprint Library:PinHeader_1x20_P2.54mm_Vertical -> (none)
- U: renamed from R8; value 100K -> (none); footprint Resistor_SMD:R_0603_1608Metric -> (none)
- U: renamed from D3; value BLUE -> (none); footprint LED_SMD:LED_0603_1608Metric -> (none)
- U: renamed from R3; value 2M -> (none); footprint Resistor_SMD:R_0603_1608Metric -> (none)
- U: renamed from U5; value MS88FS3 -> (none); footprint kien242:MS88SF3-nRF52840 -> (none)
- U: renamed from U3; value TP4054 -> (none); footprint Library:SOT-23-5 -> (none)
- U: renamed from U1; value MIC5219-3.3YM5 -> (none); footprint Library:SOT-23-5 -> (none)
- U: renamed from SW1; value RST -> (none); footprint Button_Switch_SMD:SW_SPST_B3U-1000P -> (none)
- U: renamed from C3; value 10uF -> (none); footprint Capacitor_Tantalum_SMD:CP_EIA-3216-12_Kemet-S -> (none)
- U: renamed from J1; value USB_C_Receptacle_USB2.0 -> (none); footprint kien242:USB-C-16pin-hight -> (none)
- U: renamed from R4; value 5.1k -> (none); footprint Resistor_SMD:R_0603_1608Metric -> (none)
- U: renamed from C5; value 100nF -> (none); footprint Capacitor_SMD:C_0603_1608Metric -> (none)
- U: renamed from D2; value 1N5819 -> (none); footprint Diode_SMD:D_SOD-323_HandSoldering -> (none)
- U: renamed from Q2; value AO3407 -> (none); footprint Package_TO_SOT_SMD:SOT-23 -> (none)
- U: renamed from J2; value (none) -> (none); footprint Library:PinHeader_1x20_P2.54mm_Vertical -> (none)
- U: renamed from R7; value 10M -> (none); footprint Resistor_SMD:R_0603_1608Metric -> (none)
- U: renamed from U2; value USBLC6-2SC6 -> (none); footprint Library:SOT-23-6 -> (none)
- U: renamed from R10; value 2k -> (none); footprint Resistor_SMD:R_0603_1608Metric -> (none)
- U: renamed from SW2; value DFU -> (none); footprint Button_Switch_SMD:SW_SPST_B3U-1000P -> (none)
- U: renamed from J4; value (none) -> (none); footprint TestPoint:TestPoint_Pad_1.5x1.5mm -> (none)
- U: renamed from C1; value 10nF -> (none); footprint Capacitor_SMD:C_0603_1608Metric -> (none)
- U: renamed from R1; value 2M -> (none); footprint Resistor_SMD:R_0603_1608Metric -> (none)
- U: renamed from R6; value 100K -> (none); footprint Resistor_SMD:R_0603_1608Metric -> (none)
- U: renamed from C2; value 10uF -> (none); footprint Capacitor_Tantalum_SMD:CP_EIA-3216-12_Kemet-S -> (none)
- U: renamed from R9; value 1K -> (none); footprint Resistor_SMD:R_0603_1608Metric -> (none)
Connections:
- net LED_2 is gone; now on net 0.24: U.60 (1.03)
- net 0.05: now also U.15 (Pin_15); no longer U.14 (Pin_14)
- net 0.27: now also U.14 (Pin_14); no longer U.15 (Pin_15)
- net 1.00: now also U.59 (1.01)
- net DFU: now also U.56 (0.10); no longer U.59 (1.01)
- net LED_1: now also U.2 (1.11); no longer U.58 (1.05)
- net POWER_PIN: now also U.58 (1.05)
- net SWDIO: now also U.57 (1.07)
- net 009: now reaches U.55 (0.09)
- net 009: now also U.1 (Pin_1)
- removed net 1.07: U.1 (Pin_1), U.57 (1.07)
