File: PCB/PCB/RGB.kicad_sch (KiCad schematic)
At the start: 22 parts

Commit message: cap nhat luc nua dem 23:54 12/06/2022
Parts:
- C1, C10, C2, C3, C4, C5, C6, C7, C8, C9: footprint (none) -> Capacitor_SMD:C_0603_1608Metric
Changed lines of the file:
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@@
       (effects (font (size 1.27 1.27)) (justify left))
     )
-    (property "Footprint" "" (id 2) (at 47.625 33.02 0)
+    (property "Footprint" "Capacitor_SMD:C_0603_1608Metric" (id 2) (at 47.625 33.02 0)
       (effects (font (size 1.27 1.27)) hide)
     )
@@
       (effects (font (size 1.27 1.27)) (justify left))
     )
-    (property "Footprint" "" (id 2) (at 247.65 33.02 0)
+    (property "Footprint" "Capacitor_SMD:C_0603_1608Metric" (id 2) (at 247.65 33.02 0)
       (effects (font (size 1.27 1.27)) hide)
     )
@@
       (effects (font (size 1.27 1.27)) (justify left))
     )
-    (property "Footprint" "" (id 2) (at 180.975 33.02 0)
+    (property "Footprint" "Capacitor_SMD:C_0603_1608Metric" (id 2) (at 180.975 33.02 0)
       (effects (font (size 1.27 1.27)) hide)
     )
@@
       (effects (font (size 1.27 1.27)) (justify left))
     )
-    (property "Footprint" "" (id 2) (at 136.525 33.02 0)
+    (property "Footprint" "Capacitor_SMD:C_0603_1608Metric" (id 2) (at 136.525 33.02 0)
       (effects (font (size 1.27 1.27)) hide)
     )
@@
       (effects (font (size 1.27 1.27)) (justify left))
     )
-    (property "Footprint" "" (id 2) (at 114.3 33.02 0)
+    (property "Footprint" "Capacitor_SMD:C_0603_1608Metric" (id 2) (at 114.3 33.02 0)
       (effects (font (size 1.27 1.27)) hide)
     )
@@
       (effects (font (size 1.27 1.27)) (justify left))
     )
-    (property "Footprint" "" (id 2) (at 69.85 33.02 0)
+    (property "Footprint" "Capacitor_SMD:C_0603_1608Metric" (id 2) (at 69.85 33.02 0)
       (effects (font (size 1.27 1.27)) hide)
     )
@@
       (effects (font (size 1.27 1.27)) (justify left))
     )
-    (property "Footprint" "" (id 2) (at 203.2 33.02 0)
+    (property "Footprint" "Capacitor_SMD:C_0603_1608Metric" (id 2) (at 203.2 33.02 0)
       (effects (font (size 1.27 1.27)) hide)
     )
@@
       (effects (font (size 1.27 1.27)) (justify left))
     )
-    (property "Footprint" "" (id 2) (at 158.75 33.02 0)
+    (property "Footprint" "Capacitor_SMD:C_0603_1608Metric" (id 2) (at 158.75 33.02 0)
       (effects (font (size 1.27 1.27)) hide)
     )
@@
       (effects (font (size 1.27 1.27)) (justify left))
     )
-    (property "Footprint" "" (id 2) (at 92.075 33.02 0)
+    (property "Footprint" "Capacitor_SMD:C_0603_1608Metric" (id 2) (at 92.075 33.02 0)
       (effects (font (size 1.27 1.27)) hide)
     )
@@
       (effects (font (size 1.27 1.27)) (justify left))
     )
-    (property "Footprint" "" (id 2) (at 225.425 33.02 0)
-      (effects (font (size 1.27 1.27)) hide)
-    )
+    (property "Footprint" "Capacitor_SMD:C_0603_1608Metric" (id 2) (at 225.425 33.02 0)
+      (effects (font (size 1.27 1.27)) hide)
+    )

Commit message: cap nhat 11:55 13/06/2022
Parts:
- added C11, C12, C13, C14, C15, C16, C17, C18, C19, C20: 104, Capacitor_SMD:C_0603_1608Metric, symbol Device:C_Small
Connections:
- net +3V3: now also C11.1, C12.1, C13.1, C14.1, C15.1, C16.1, C17.1, C18.1, C19.1, C20.1
- net GND: now also C11.2, C12.2, C13.2, C14.2, C15.2, C16.2, C17.2, C18.2, C19.2, C20.2

Commit message: Cập nhật 22:10 18/06/2022
Parts:
- added J14, J15, J28, J29: (no value), Library:Conn_01x01, symbol Connector_Generic:Conn_01x01
Connections:
- net RGB_PROMICRO: now also J14.1 (Pin_1), J15.1 (Pin_1)
- net at JP10.2 (B), JP9.2 (B), LED7.O (OUT)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: now also J28.1 (Pin_1), J29.1 (Pin_1)
Changed lines of the file:
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@@
   (junction (at 225.425 45.72) (diameter 0) (color 0 0 0 0)
   )
+  (junction (at 186.055 66.04) (diameter 0) (color 0 0 0 0)
+  )
   (junction (at 92.075 30.48) (diameter 0) (color 0 0 0 0)
   )
@@
   (junction (at 82.55 30.48) (diameter 0) (color 0 0 0 0)
   )
+  (junction (at 99.695 66.04) (diameter 0) (color 0 0 0 0)
+  )
   (junction (at 47.625 45.72) (diameter 0) (color 0 0 0 0)
   )
@@
     (stroke (width 0) (type default) (color 0 0 0 0))
   )
-  (wire (pts (xy 132.08 66.04) (xy 97.155 66.04))
+  (wire (pts (xy 132.08 66.04) (xy 99.695 66.04))
     (stroke (width 0) (type default) (color 0 0 0 0))
   )
@@
   )
   (wire (pts (xy 180.975 45.72) (xy 171.45 45.72))
+    (stroke (width 0) (type default) (color 0 0 0 0))
+  )
+  (wire (pts (xy 99.695 66.04) (xy 97.155 66.04))
     (stroke (width 0) (type default) (color 0 0 0 0))
   )
@@
     )
   )
+  (symbol (lib_id "Connector_Generic:Conn_01x01") (at 99.695 71.12 270) (unit 1)
+    (in_bom yes) (on_board yes)
+    (property "Reference" "J14" (id 0) (at 99.695 71.12 0))
+    (property "Value" " " (id 1) (at 95.885 71.12 0))
+    (property "Footprint" "Library:Conn_01x01" (id 2) (at 99.695 71.12 0)
+      (effects (font (size 1.27 1.27)) hide)
+    )
+    (property "Datasheet" "~" (id 3) (at 99.695 71.12 0)
+      (effects (font (size 1.27 1.27)) hide)
+    )
+    (pin "1")
+  )
   (symbol (lib_id "Device:C_Small") (at 47.625 33.02 0) (unit 1)
     (in_bom yes) (on_board yes)
@@
     (pin "1")
     (pin "2")
+  )
+  (symbol (lib_id "Connector_Generic:Conn_01x01") (at 99.695 71.12 270) (unit 1)
+    (in_bom yes) (on_board yes)
+    (property "Reference" "J15" (id 0) (at 99.695 71.12 0))
+    (property "Value" " " (id 1) (at 95.885 71.12 0))
+    (property "Footprint" "Library:Conn_01x01" (id 2) (at 99.695 71.12 0)
+      (effects (font (size 1.27 1.27)) hide)
+    )
+    (property "Datasheet" "~" (id 3) (at 99.695 71.12 0)
+      (effects (font (size 1.27 1.27)) hide)
+    )
+    (pin "1")
   )
   (symbol (lib_id "power:GND") (at 95.885 88.265 0) (unit 1)
@@
     (pin "2")
   )
+  (symbol (lib_id "Connector_Generic:Conn_01x01") (at 186.055 71.12 270) (unit 1)
+    (in_bom yes) (on_board yes)
+    (property "Reference" "J28" (id 0) (at 186.055 71.12 0))
+    (property "Value" " " (id 1) (at 182.245 71.12 0))
+    (property "Footprint" "Library:Conn_01x01" (id 2) (at 186.055 71.12 0)
+      (effects (font (size 1.27 1.27)) hide)
+    )
+    (property "Datasheet" "~" (id 3) (at 186.055 71.12 0)
+      (effects (font (size 1.27 1.27)) hide)
+    )
+    (pin "1")
+  )
   (symbol (lib_id "kien242:6812") (at 193.675 38.1 0) (unit 1)
     (in_bom yes) (on_board yes)
@@
       (effects (font (size 1.27 1.27)) hide)
     )
+    (pin "1")
+  )
+  (symbol (lib_id "Connector_Generic:Conn_01x01") (at 186.055 71.12 270) (unit 1)
+    (in_bom yes) (on_board yes)
+    (property "Reference" "J29" (id 0) (at 186.055 71.12 0))
+    (property "Value" " " (id 1) (at 182.245 71.12 0))
+    (property "Footprint" "Library:Conn_01x01" (id 2) (at 186.055 71.12 0)
+      (effects (font (size 1.27 1.27)) hide)
+    )
+    (property "Datasheet" "~" (id 3) (at 186.055 71.12 0)
+      (effects (font (size 1.27 1.27)) hide)
+    )
