File: PCB/PCB/SofleKeyboard.kicad_sch (KiCad schematic)
At the start: 115 parts, among them J1 DATA Port, J2 DATA Port, J3 Conn_01x04, J4 , SW1 1u, SW10 1u, SW11 1u, SW12 1u, SW13 1u, SW14 1u, SW15 1u, SW16 1u, SW17 1u, SW18 1u, SW19 1u, SW2 1u, SW20 1u, SW21 1u, SW22 1u, SW23 1u, SW24 1u, SW25 1u, SW26 1u, SW27 1u, SW28 1u, SW29 1u, SW3 1u, SW30 1u, SW31 , SW32 1u, SW33 1u, SW34 1u, SW35 1u, SW36 1u, SW37 1u, SW38 1u, SW39 1u, SW4 1u, SW40 1u, SW41 1u, SW42 1u, SW43 1u, SW44 1u, SW45 1u, SW46 1.5u, SW47 , SW48 , SW5 1u, SW6 1u, SW7 1u, SW8 1u, SW9 1u, U1 Promicro, U2 Blackpill-F4x1

Commit message: cap nhat luc nua dem 23:54 12/06/2022
Parts:
- added R1, R2: 10k, Resistor_SMD:R_0603_1608Metric, symbol Device:R
Connections:
- net +3V3: now also R1.1, R2.1
- net RX: now also R1.2
- net TX: now also R2.2
Changed lines of the file:
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@@
+    )
+  )
+  (global_label "RX" (shape input) (at 57.15 99.06 270) (fields_autoplaced)
+    (effects (font (size 1.27 1.27)) (justify right))
+    (property "Intersheet References" "${INTERSHEET_REFS}" (id 0) (at 57.2294 103.8637 90)
+      (effects (font (size 1.27 1.27)) (justify right) hide)
     )
   )
@@
     (property "Intersheet References" "${INTERSHEET_REFS}" (id 0) (at 69.215 -59.055 90)
       (effects (font (size 1.27 1.27)) (justify left) hide)
+    )
+  )
+  (global_label "TX" (shape input) (at 63.5 99.06 270) (fields_autoplaced)
+    (effects (font (size 1.27 1.27)) (justify right))
+    (property "Intersheet References" "${INTERSHEET_REFS}" (id 0) (at 63.5794 103.5613 90)
+      (effects (font (size 1.27 1.27)) (justify right) hide)
     )
   )
@@
     (pin "2")
   )
+  (symbol (lib_id "power:+3.3V") (at 57.15 91.44 0) (unit 1)
+    (in_bom yes) (on_board yes) (fields_autoplaced)
+    (property "Reference" "#PWR0109" (id 0) (at 57.15 95.25 0)
+      (effects (font (size 1.27 1.27)) hide)
+    )
+    (property "Value" "+3.3V" (id 1) (at 57.15 86.36 0))
+    (property "Footprint" "" (id 2) (at 57.15 91.44 0)
+      (effects (font (size 1.27 1.27)) hide)
+    )
+    (property "Datasheet" "" (id 3) (at 57.15 91.44 0)
+      (effects (font (size 1.27 1.27)) hide)
+    )
+    (pin "1")
+  )
+  (symbol (lib_id "Device:R") (at 63.5 95.25 0) (unit 1)
+    (in_bom yes) (on_board yes)
+    (property "Reference" "R2" (id 0) (at 64.135 92.075 0)
+      (effects (font (size 1.27 1.27)) (justify left))
+    )
+    (property "Value" "10k" (id 1) (at 63.5 97.155 90)
+      (effects (font (size 1.27 1.27)) (justify left))
+    )
+    (property "Footprint" "Resistor_SMD:R_0603_1608Metric" (id 2) (at 61.722 95.25 90)
+      (effects (font (size 1.27 1.27)) hide)
+    )
+    (property "Datasheet" "~" (id 3) (at 63.5 95.25 0)
+      (effects (font (size 1.27 1.27)) hide)
+    )
+    (pin "1")
+    (pin "2")
+  )
   (symbol (lib_id "SofleKeyboard-rescue:SW_PUSH-Lily58-cache-Lily58_Pro-rescue") (at 66.04 58.42 0) (mirror y) (unit 1)
     (in_bom yes) (on_board yes)
@@
     )
     (property "Datasheet" "" (id 3) (at 38.1 62.23 0)
+      (effects (font (size 1.27 1.27)) hide)
+    )
+    (pin "1")
+    (pin "2")
+  )
+  (symbol (lib_id "Device:R") (at 57.15 95.25 0) (unit 1)
+    (in_bom yes) (on_board yes)
+    (property "Reference" "R1" (id 0) (at 57.785 92.075 0)
+      (effects (font (size 1.27 1.27)) (justify left))
+    )
+    (property "Value" "10k" (id 1) (at 57.15 97.155 90)
+      (effects (font (size 1.27 1.27)) (justify left))
+    )
+    (property "Footprint" "Resistor_SMD:R_0603_1608Metric" (id 2) (at 55.372 95.25 90)
+      (effects (font (size 1.27 1.27)) hide)
+    )
+    (property "Datasheet" "~" (id 3) (at 57.15 95.25 0)
       (effects (font (size 1.27 1.27)) hide)
     )
@@
     (pin "1")
     (pin "2")
+  )
+  (symbol (lib_id "power:+3.3V") (at 63.5 91.44 0) (unit 1)
+    (in_bom yes) (on_board yes) (fields_autoplaced)
+    (property "Reference" "#PWR0108" (id 0) (at 63.5 95.25 0)
+      (effects (font (size 1.27 1.27)) hide)
+    )
+    (property "Value" "+3.3V" (id 1) (at 63.5 86.36 0))
+    (property "Footprint" "" (id 2) (at 63.5 91.44 0)
+      (effects (font (size 1.27 1.27)) hide)
+    )
+    (property "Datasheet" "" (id 3) (at 63.5 91.44 0)
+      (effects (font (size 1.27 1.27)) hide)
+    )
+    (pin "1")
   )
   (symbol (lib_id "Jumper:SolderJumper_2_Open") (at 241.935 132.715 0) (unit 1)
@@
       (reference "#PWR0107") (unit 1) (value "+3.3V") (footprint "")
     )
+    (path "/b590eaca-09b6-4a9c-bf06-133b1d153b35"
+      (reference "#PWR0108") (unit 1) (value "+3.3V") (footprint "")
+    )
+    (path "/4107ae43-ef7b-4881-bf28-19412946e234"
+      (reference "#PWR0109") (unit 1) (value "+3.3V") (footprint "")
+    )
     (path "/d5f0102a-ccd2-481d-aac9-a500663069d8/0d44eaf9-a0c8-43b4-a607-55aa510fbbda"
-      (reference "C1") (unit 1) (value "104") (footprint "")
+      (reference "C1") (unit 1) (value "104") (footprint "Capacitor_SMD:C_0603_1608Metric")
     )
     (path "/d5f0102a-ccd2-481d-aac9-a500663069d8/887417aa-cab8-43aa-a3d3-197eaed6ffeb"
-      (reference "C2") (unit 1) (value "104") (footprint "")
+      (reference "C2") (unit 1) (value "104") (footprint "Capacitor_SMD:C_0603_1608Metric")
     )
     (path "/d5f0102a-ccd2-481d-aac9-a500663069d8/d7ea459a-dc44-44d8-bb2b-fa117592f2ce"
-      (reference "C3") (unit 1) (value "104") (footprint "")
+      (reference "C3") (unit 1) (value "104") (footprint "Capacitor_SMD:C_0603_1608Metric")
     )
     (path "/d5f0102a-ccd2-481d-aac9-a500663069d8/7f4e2763-9eaf-403f-a259-43cdce5d501c"
-      (reference "C4") (unit 1) (value "104") (footprint "")
+      (reference "C4") (unit 1) (value "104") (footprint "Capacitor_SMD:C_0603_1608Metric")
     )
     (path "/d5f0102a-ccd2-481d-aac9-a500663069d8/562f6c0a-b067-4aa0-b5e1-f2069e4e9a0c"
-      (reference "C5") (unit 1) (value "104") (footprint "")
+      (reference "C5") (unit 1) (value "104") (footprint "Capacitor_SMD:C_0603_1608Metric")
     )
     (path "/d5f0102a-ccd2-481d-aac9-a500663069d8/be10c843-ddcd-4be2-a400-b25bbc99f1c2"
-      (reference "C6") (unit 1) (value "104") (footprint "")
+      (reference "C6") (unit 1) (value "104") (footprint "Capacitor_SMD:C_0603_1608Metric")
     )
     (path "/d5f0102a-ccd2-481d-aac9-a500663069d8/487338e1-08d8-4e08-8493-e7c5f4aaefef"
-      (reference "C7") (unit 1) (value "104") (footprint "")
+      (reference "C7") (unit 1) (value "104") (footprint "Capacitor_SMD:C_0603_1608Metric")
     )
     (path "/d5f0102a-ccd2-481d-aac9-a500663069d8/b6a8f8b1-cf05-4426-8b0c-4a39c90b89c1"
-      (reference "C8") (unit 1) (value "104") (footprint "")
+      (reference "C8") (unit 1) (value "104") (footprint "Capacitor_SMD:C_0603_1608Metric")
     )
     (path "/d5f0102a-ccd2-481d-aac9-a500663069d8/f5652ad8-ac94-4a27-940a-aa1b8772e379"
-      (reference "C9") (unit 1) (value "104") (footprint "")
+      (reference "C9") (unit 1) (value "104") (footprint "Capacitor_SMD:C_0603_1608Metric")
     )
     (path "/d5f0102a-ccd2-481d-aac9-a500663069d8/23cef0b6-aead-42d9-8935-e695feb97274"
-      (reference "C10") (unit 1) (value "104") (footprint "")
+      (reference "C10") (unit 1) (value "104") (footprint "Capacitor_SMD:C_0603_1608Metric")
     )
     (path "/91aa030c-cd7a-4bf6-a3e6-bccd5e0d552c"
@@
       (reference "LED10") (unit 1) (value "6812") (footprint "kien242:SK6812MINI-FLIP")
     )
+    (path "/633aafcb-e7f5-4f49-b90e-2af365a07e52"
+      (reference "R1") (unit 1) (value "10k") (footprint "Resistor_SMD:R_0603_1608Metric")
+    )
+    (path "/47bef882-7796-4249-9d91-9e6b1c94b8bb"
+      (reference "R2") (unit 1) (value "10k") (footprint "Resistor_SMD:R_0603_1608Metric")
+    )
     (path "/e7dfaf12-5663-403e-b5a3-586865df3607"

Commit message: cap nhat 11:55 13/06/2022
Parts:
- R1, R2: footprint Resistor_SMD:R_0603_1608Metric -> Library:R_0805_2012Metric_Pad1.20x1.40mm_HandSolder
Changed lines of the file:
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@@
       (effects (font (size 1.27 1.27)) (justify left))
     )
-    (property "Footprint" "Resistor_SMD:R_0603_1608Metric" (id 2) (at 61.722 95.25 90)
+    (property "Footprint" "Library:R_0805_2012Metric_Pad1.20x1.40mm_HandSolder" (id 2) (at 61.722 95.25 90)
       (effects (font (size 1.27 1.27)) hide)
     )
@@
       (effects (font (size 1.27 1.27)) (justify left))
     )
-    (property "Footprint" "Resistor_SMD:R_0603_1608Metric" (id 2) (at 55.372 95.25 90)
+    (property "Footprint" "Library:R_0805_2012Metric_Pad1.20x1.40mm_HandSolder" (id 2) (at 55.372 95.25 90)
       (effects (font (size 1.27 1.27)) hide)
     )
@@
       (reference "#PWR0109") (unit 1) (value "+3.3V") (footprint "")
     )
+    (path "/d5f0102a-ccd2-481d-aac9-a500663069d8/de2ae919-ef2c-4c13-b65e-4e2417e55785"
+      (reference "#PWR0110") (unit 1) (value "+3.3V") (footprint "")
+    )
+    (path "/d5f0102a-ccd2-481d-aac9-a500663069d8/c0a34e97-87d6-47e8-a2c2-8827172c43ef"
+      (reference "#PWR0111") (unit 1) (value "+3.3V") (footprint "")
+    )
+    (path "/d5f0102a-ccd2-481d-aac9-a500663069d8/c4dab5f1-5786-46db-ab7a-1b44fd1dd33c"
+      (reference "#PWR0112") (unit 1) (value "+3.3V") (footprint "")
+    )
+    (path "/d5f0102a-ccd2-481d-aac9-a500663069d8/1a2cbb7d-a12b-4ce2-8cb5-723dbf106184"
+      (reference "#PWR0113") (unit 1) (value "GND") (footprint "")
+    )
+    (path "/d5f0102a-ccd2-481d-aac9-a500663069d8/ea622771-3cf0-4c6c-863e-6326c4f96725"
+      (reference "#PWR0114") (unit 1) (value "+3.3V") (footprint "")
+    )
+    (path "/d5f0102a-ccd2-481d-aac9-a500663069d8/2eec7e7a-4330-4f6e-9016-3a7281b4315e"
+      (reference "#PWR0115") (unit 1) (value "GND") (footprint "")
+    )
+    (path "/d5f0102a-ccd2-481d-aac9-a500663069d8/dc7ffb7f-ab71-4bf8-9657-248abbf0d595"
+      (reference "#PWR0116") (unit 1) (value "+3.3V") (footprint "")
+    )
+    (path "/d5f0102a-ccd2-481d-aac9-a500663069d8/cd0c9c20-e15d-4fe8-86ae-a7aa89b66ad5"
+      (reference "#PWR0117") (unit 1) (value "GND") (footprint "")
+    )
+    (path "/d5f0102a-ccd2-481d-aac9-a500663069d8/239ba5d9-a1e7-472b-9463-5fd60ba27aec"
+      (reference "#PWR0118") (unit 1) (value "+3.3V") (footprint "")
+    )
+    (path "/d5f0102a-ccd2-481d-aac9-a500663069d8/e05ab311-16ee-4afe-afba-54842d71dc7d"
+      (reference "#PWR0119") (unit 1) (value "GND") (footprint "")
+    )
+    (path "/d5f0102a-ccd2-481d-aac9-a500663069d8/2ce8521d-b4f6-41fe-a3f6-e943f0a06d49"
+      (reference "#PWR0120") (unit 1) (value "+3.3V") (footprint "")
+    )
+    (path "/d5f0102a-ccd2-481d-aac9-a500663069d8/85636cb1-c8ea-4762-a108-8c9d6362caf3"
+      (reference "#PWR0121") (unit 1) (value "GND") (footprint "")
+    )
+    (path "/d5f0102a-ccd2-481d-aac9-a500663069d8/5de4fbb2-1b94-40fa-a7eb-5ad36fe8b0cd"
+      (reference "#PWR0122") (unit 1) (value "GND") (footprint "")
+    )
+    (path "/d5f0102a-ccd2-481d-aac9-a500663069d8/bd24c0cc-ba9e-4303-87ac-871ef5acb4de"
+      (reference "#PWR0123") (unit 1) (value "+3.3V") (footprint "")
+    )
+    (path "/d5f0102a-ccd2-481d-aac9-a500663069d8/9e7456c4-7fc3-45aa-88a0-82140af05094"
+      (reference "#PWR0124") (unit 1) (value "GND") (footprint "")
+    )
+    (path "/d5f0102a-ccd2-481d-aac9-a500663069d8/3edb8056-dfbd-4dc3-b4f3-1a443b05e4c3"
+      (reference "#PWR0125") (unit 1) (value "GND") (footprint "")
+    )
+    (path "/d5f0102a-ccd2-481d-aac9-a500663069d8/d5d32a32-b3bf-455c-a349-308eaf785aff"
+      (reference "#PWR0126") (unit 1) (value "GND") (footprint "")
+    )
+    (path "/d5f0102a-ccd2-481d-aac9-a500663069d8/c0a2fe72-5e38-4b73-93ef-62b27577e2dc"
+      (reference "#PWR0127") (unit 1) (value "GND") (footprint "")
+    )
+    (path "/d5f0102a-ccd2-481d-aac9-a500663069d8/623a95d3-92aa-43fc-bfb7-1927169d4600"
+      (reference "#PWR0128") (unit 1) (value "+3.3V") (footprint "")
+    )
+    (path "/d5f0102a-ccd2-481d-aac9-a500663069d8/d0eb2768-bb97-4e38-bc3c-5e38821b161a"
+      (reference "#PWR0129") (unit 1) (value "+3.3V") (footprint "")
+    )
     (path "/d5f0102a-ccd2-481d-aac9-a500663069d8/0d44eaf9-a0c8-43b4-a607-55aa510fbbda"
       (reference "C1") (unit 1) (value "104") (footprint "Capacitor_SMD:C_0603_1608Metric")
@@
       (reference "C10") (unit 1) (value "104") (footprint "Capacitor_SMD:C_0603_1608Metric")
     )
+    (path "/d5f0102a-ccd2-481d-aac9-a500663069d8/f7a08f47-28a3-4664-b73f-efd412909c91"
+      (reference "C11") (unit 1) (value "104") (footprint "Capacitor_SMD:C_0603_1608Metric")
+    )
+    (path "/d5f0102a-ccd2-481d-aac9-a500663069d8/3fc5f0c6-b153-4d2b-a97b-280ebd06937c"
+      (reference "C12") (unit 1) (value "104") (footprint "Capacitor_SMD:C_0603_1608Metric")
+    )
+    (path "/d5f0102a-ccd2-481d-aac9-a500663069d8/3ad3e90c-da30-40da-b83d-347234a4d46b"
+      (reference "C13") (unit 1) (value "104") (footprint "Capacitor_SMD:C_0603_1608Metric")
+    )
+    (path "/d5f0102a-ccd2-481d-aac9-a500663069d8/daa113bb-7151-408c-9a5d-9fc0742a8799"
+      (reference "C14") (unit 1) (value "104") (footprint "Capacitor_SMD:C_0603_1608Metric")
+    )
+    (path "/d5f0102a-ccd2-481d-aac9-a500663069d8/f77e1cf1-10b8-41d1-9804-feb0bc1d2b6c"
+      (reference "C15") (unit 1) (value "104") (footprint "Capacitor_SMD:C_0603_1608Metric")
+    )
+    (path "/d5f0102a-ccd2-481d-aac9-a500663069d8/c8c3ba6e-6f6e-4a97-b351-bbff9b9bdcc2"
+      (reference "C16") (unit 1) (value "104") (footprint "Capacitor_SMD:C_0603_1608Metric")
+    )
+    (path "/d5f0102a-ccd2-481d-aac9-a500663069d8/4d8f03af-088e-4619-bd96-718d9784eab5"
+      (reference "C17") (unit 1) (value "104") (footprint "Capacitor_SMD:C_0603_1608Metric")
+    )
+    (path "/d5f0102a-ccd2-481d-aac9-a500663069d8/f2c834f9-c103-4334-8883-5d3b18f11be6"
+      (reference "C18") (unit 1) (value "104") (footprint "Capacitor_SMD:C_0603_1608Metric")
+    )
+    (path "/d5f0102a-ccd2-481d-aac9-a500663069d8/e1581e33-26a5-41d6-8d99-da00ff6956c5"
+      (reference "C19") (unit 1) (value "104") (footprint "Capacitor_SMD:C_0603_1608Metric")
+    )
+    (path "/d5f0102a-ccd2-481d-aac9-a500663069d8/40c4c9f9-f780-4cff-b616-381fe6ca3a50"
+      (reference "C20") (unit 1) (value "104") (footprint "Capacitor_SMD:C_0603_1608Metric")
+    )
     (path "/91aa030c-cd7a-4bf6-a3e6-bccd5e0d552c"
       (reference "D1") (unit 1) (value "D") (footprint "Library:Diode")
@@
     )
     (path "/633aafcb-e7f5-4f49-b90e-2af365a07e52"
-      (reference "R1") (unit 1) (value "10k") (footprint "Resistor_SMD:R_0603_1608Metric")
+      (reference "R1") (unit 1) (value "10k") (footprint "Library:R_0805_2012Metric_Pad1.20x1.40mm_HandSolder")
     )
     (path "/47bef882-7796-4249-9d91-9e6b1c94b8bb"
-      (reference "R2") (unit 1) (value "10k") (footprint "Resistor_SMD:R_0603_1608Metric")
+      (reference "R2") (unit 1) (value "10k") (footprint "Library:R_0805_2012Metric_Pad1.20x1.40mm_HandSolder")
     )
     (path "/e7dfaf12-5663-403e-b5a3-586865df3607"

Commit message: 18:29 13/06/2022
Parts:
- added H1, H2, H3, H6: Hole, Library:Cut_hole, symbol keebio:Hole
- SW11, SW12: footprint Library:SW-HS-Flip-1u -> Library:SW-HS_flip-1u
- SW13, SW14: footprint Library:SW-HS_flip-1u -> Library:SW-HS-Flip-1u
Connections:
- net +3V3: no longer U1.D4
- net RGB_PROMICRO: now also U1.F6; no longer U1.E6
- net col0': now also U1.B3 ((MISO)B3); no longer U1.D3 (D3(TX))
- net col1': now also SW2.2, U1.B2 ((MOSI)B2); no longer SW2.1, U1.C6, U1.F7
- net col2': now also U1.E6; no longer U1.B5
- net col3': now also U1.D1 (D1(SDA)), U1.F4, U1.F5; no longer U1.B4
- net row0: now also U1.F7; no longer U1.D2 (D2(RX))
- net row1: now also U1.D4; no longer U1.F4
- net row2: now also U1.B5; no longer U1.B2 ((MOSI)B2)
- net row3: now also U1.B4; no longer U1.B6
- net at D2.2 (A): now also SW2.1; no longer SW2.2

Commit message: Cập nhật 22:10 18/06/2022
Parts:
- removed D1, D11, D21, D31: D, Library:Diode, symbol SofleKeyboard-rescue:D-Lily58-cache-Lily58_Pro-rescue
- removed SW1, SW11, SW21, SW32: 1u, Library:SW-HS_flip-1u, symbol SofleKeyboard-rescue:SW_PUSH-Lily58-cache-Lily58_Pro-rescue
- added J10, J11, J12, J13, J16, J17, J18, J19, J20, J21, J22, J23, J24, J25, J26, J27, J6, J7, J8, J9: (no value), Library:Conn_01x01, symbol Connector_Generic:Conn_01x01
- added J5: Conn_01x08, Library:Conn_01x08, symbol Connector_Generic:Conn_01x08
- added TH10, TH9: HOLE, Library:M2_HOLE_PCB, symbol SofleKeyboard-rescue:HOLE-Lily58-cache-Lily58_Pro-rescue
Connections:
- net +3V3: now also J24.1 (Pin_1), J25.1 (Pin_1), J26.1 (Pin_1), J27.1 (Pin_1); no longer JP2.1 (A), JP7.1 (A), R1.1, R2.1, U2.23 (3.3V), U2.5 (PA8)
- net ENCA: now also U2.34 (PA1); no longer U2.30 (PA5)
- net ENCB: now also U2.35 (PA0); no longer U2.31 (PA4)
- net GND: now also J16.1 (Pin_1), J17.1 (Pin_1), J5.8 (Pin_8)
- net col0': no longer U1.B3 ((MISO)B3)
- net col1': now also J18.1 (Pin_1), J19.1 (Pin_1)
- net col2': now also J20.1 (Pin_1), J21.1 (Pin_1)
- net col3': now also J22.1 (Pin_1), J23.1 (Pin_1)
- net row0: now also U2.5 (PA8), J6.1 (Pin_1), J7.1 (Pin_1); no longer U2.4 (PB15)
- net row1: now also J8.1 (Pin_1), J9.1 (Pin_1)
- net row2: now also U2.4 (PB15), J10.1 (Pin_1), J11.1 (Pin_1); no longer U2.27 (PB0)
- net row3: now also U2.3 (PB14), J12.1 (Pin_1), J13.1 (Pin_1); no longer U2.28 (PA7)
- net row4: now also U2.31 (PA4); no longer U2.29 (PA6)
- net DC: now reaches U2.24 (PB10)
- net DC: now also J5.3 (Pin_3)
- net CS: now reaches U2.26 (PB1)
- net CS: now also J5.2 (Pin_2)
- net RES: now reaches U2.39 (PC13)
- net RES: now also J5.4 (Pin_4)
- new net 3.3_TOP: J5.7 (Pin_7), JP2.1 (A), JP7.1 (A), R1.1, R2.1, U2.23 (3.3V)
- new net BLK: J5.1 (Pin_1), U2.27 (PB0)
- new net MOSI: J5.5 (Pin_5), U2.28 (PA7)
- new net SCK: J5.6 (Pin_6), U2.30 (PA5)
Other:
- moved on the sheet: R1, R2
