File: PCB/lmao/RGB.kicad_sch (KiCad schematic)
At the start: 54 parts

Commit message: Cập nhật Lmao
Parts:
- C10, C11, C12, C13, C14, C15, C16, C17, C18, C19, C20, C21, C22, C23, C24, C25, C26, C27, C28, C29, C30, C31, C32, C33, C34, C35, C9: value (none) -> C; footprint (none) -> Capacitor_SMD:C_0603_1608Metric_Pad1.08x0.95mm_HandSolder
- LED1, LED10, LED11, LED12, LED13, LED14, LED15, LED16, LED17, LED18, LED19, LED2, LED20, LED21, LED22, LED23, LED24, LED25, LED26, LED27, LED3, LED4, LED5, LED6, LED7, LED8, LED9: value (none) -> 6812; footprint (none) -> kien242:SK6812-MINI

Commit message: update
Parts:
- renumbered C13 to C10, C14 to C11, C15 to C12, C16 to C13, C17 to C14, C18 to C15, C19 to C16, C20 to C17, C21 to C18, C22 to C19, C23 to C20, C24 to C21, C25 to C22, C26 to C23, C27 to C24, C28 to C25, C29 to C26, C30 to C27, C31 to C28, C32 to C29, C33 to C30, C34 to C31, C35 to C32, C9 to C6, C10 to C7, C11 to C8, C12 to C9, LED4 to LED10, LED13 to LED11, LED22 to LED12, LED5 to LED13, LED23 to LED15, LED6 to LED16, LED15 to LED17, LED24 to LED18, LED7 to LED19, LED10 to LED2, LED16 to LED20, LED25 to LED21, LED8 to LED22, LED17 to LED23, LED26 to LED24, LED9 to LED25, LED18 to LED26, LED19 to LED3, LED2 to LED4, LED11 to LED5, LED20 to LED6, LED3 to LED7, LED12 to LED8, LED21 to LED9

Commit message: update Lmao keyboard
Parts:
- renumbered LED2 to LED10, LED5 to LED11, LED8 to LED12, LED11 to LED13, LED17 to LED15, LED20 to LED16, LED23 to LED17, LED26 to LED18, LED3 to LED19, LED4 to LED2, LED6 to LED20, LED9 to LED21, LED12 to LED22, LED15 to LED23, LED18 to LED24, LED21 to LED25, LED24 to LED26, LED7 to LED3, LED10 to LED4, LED13 to LED5, LED16 to LED6, LED19 to LED7, LED22 to LED8, LED25 to LED9
