File: PCB/lmao/lmao.kicad_pcb (KiCad board)
At the start: 2 copper layers, 243.1 x 105 mm, 58 parts, among them SW1 SW_Push, SW10 SW_Push, SW11 SW_Push, SW12 SW_Push, SW13 SW_Push, SW14 SW_Push, SW15 SW_Push, SW16 SW_Push, SW17 SW_Push, SW18 SW_Push, SW19 SW_Push, SW2 SW_Push, SW20 SW_Push, SW21 SW_Push, SW22 SW_Push, SW23 SW_Push, SW24 SW_Push, SW25 SW_Push, SW26 SW_Push, SW27 SW_Push, SW28 SW_Push, SW29 SW_Push, SW3 SW_Push, SW30 SW_Push, SW31 SW_Push, SW32 SW_Push, SW33 SW_Push, SW34 SW_Push, SW35 SW_Push, SW36 SW_Push, SW37 SW_Push, SW38 SW_Push, SW39 SW_Push, SW4 SW_Push, SW40 SW_Push, SW41 SW_Push, SW42 SW_Push, SW43 SW_Push, SW44 SW_Push, SW45 SW_Push, SW46 SW_Push, SW47 SW_Push, SW48 SW_Push, SW49 SW_Push, SW5 SW_Push, SW50 SW_Push, SW51 SW_Push, SW52 SW_Push, SW53 SW_Push, SW54 SW_Push, SW55 SW_Push, SW6 SW_Push, SW7 SW_Push, SW8 SW_Push, SW9 SW_Push

Commit message: Update Lmao
Parts:
- removed ST36, ST50, ST52: MountingHole, Stabilizer_Cherry_MX_2u
- removed SW1, SW28, SW40: SW_Push, SW_Cherry_MX_PCB_1.00u
- removed SW52: SW_Push, SW_Cherry_MX_PCB_2.25u
- removed SW53: SW_Push, SW_Cherry_MX_PCB_1.25u
- added H1: Stab, kien242:Stab, F.Cu at (48.7, 98.7)
- added H2: Stab, kien242:Stab, F.Cu at (117.8, 117.8)
- added H3: Stab, kien242:Stab, F.Cu at (177.3, 117.8)
- added J2: USB_C_Receptacle_USB2.0, kien242:USB-C-16pin-hight-v2, B.Cu at (45.7, 23.5)
- added R2: 5.1k, Resistor_SMD:R_0603_1608Metric_Pad0.98x0.95mm_HandSolder, B.Cu at (43.4, 34.8)
- added R4: 5.1k, Resistor_SMD:R_0603_1608Metric_Pad0.98x0.95mm_HandSolder, B.Cu at (48.8, 30.5)
- added SW56: 2u, MX-hotswap:SW-HS-2u, F.Cu at (117.8, 117.8)
- added SW57: 1u, MX-hotswap:SW-HS-1u, F.Cu at (146.4, 117.8)
- added SW58: 2.25u, MX-hotswap:SW-HS-2.25u, F.Cu at (177.3, 117.8)
- added SW60: 1.25u, MX-hotswap:SW-HS-1.25u, F.Cu at (210.7, 117.8)
- added SW61: 1u, MX-hotswap:SW-HS-1u, F.Cu at (232.1, 117.8)
- added SW62: 1.25u, MX-hotswap:SW-HS-1.25u, F.Cu at (253.5, 117.8)
- added U2: USBLC6-2SC6, Package_TO_SOT_SMD:SOT-23-6_Handsoldering, B.Cu at (50.5, 39.8)
- added U4: MS88FS3, kien242:MS88SF3-nRF52840, B.Cu at (255.9, 47.0)
- SW10, SW11, SW12, SW14, SW16, SW17, SW18, SW19, SW20, SW21, SW22, SW23, SW24, SW26, SW29, SW3, SW30, SW31, SW32, SW33, SW34, SW37, SW4, SW41, SW42, SW43, SW44, SW45, SW5, SW6, SW7, SW8, SW9: value SW_Push -> 1u; footprint SW_Cherry_MX_PCB_1.00u -> MX-hotswap:SW-HS-1u
- SW13: value SW_Push -> 1u; footprint SW_Cherry_MX_PCB_1.50u -> MX-hotswap:SW-HS-1u
- SW15: value SW_Push -> 1.5u; footprint SW_Cherry_MX_PCB_1.00u -> MX-hotswap:SW-HS-1.5u
- SW2: value SW_Push -> (none); footprint SW_Cherry_MX_PCB_1.00u -> kien242:MSS22D18; moved to B.Cu
- SW25, SW35: value SW_Push -> 1u; footprint SW_Cherry_MX_PCB_1.75u -> MX-hotswap:SW-HS-1u
- SW27, SW38: value SW_Push -> 1.75u; footprint SW_Cherry_MX_PCB_1.00u -> MX-hotswap:SW-HS-1.75u
- SW36: value SW_Push -> 1u; footprint SW_Cherry_MX_PCB_2.25u -> MX-hotswap:SW-HS-1u
- SW39: value SW_Push -> 2.25u; footprint SW_Cherry_MX_PCB_1.00u -> MX-hotswap:SW-HS-2.25u
- SW46, SW47, SW48, SW49: value SW_Push -> 1u; footprint SW_Cherry_MX_PCB_1.25u -> MX-hotswap:SW-HS-1u
- SW50: value SW_Push -> 1.25u; footprint SW_Cherry_MX_PCB_2.00u -> MX-hotswap:SW-HS-1.25u
- SW51, SW54: value SW_Push -> 1.25u; footprint SW_Cherry_MX_PCB_1.00u -> MX-hotswap:SW-HS-1.25u
- SW55: value SW_Push -> 1.25u; footprint SW_Cherry_MX_PCB_1.25u -> MX-hotswap:SW-HS-1.25u
- moved SW13 197.4 mm to (236.9, 36.8)
- moved SW25 194.4 mm to (236.9, 60.6)
- moved SW14 192.7 mm to (255.9, 36.8)
- moved SW26 187.3 mm to (255.9, 60.6)
- moved SW54 168.8 mm to (63.0, 117.8)
- moved SW55 166.4 mm to (86.8, 117.8)
- moved SW36 156.6 mm to (203.5, 79.7)
- moved SW47 156.6 mm to (194.0, 98.7)
- moved SW38 151.9 mm to (248.8, 79.7)
- moved SW48 151.9 mm to (213.0, 98.7)
- moved SW49 147.2 mm to (232.1, 98.7)
- moved SW37 144.9 mm to (222.6, 79.7)
- moved SW50 137.8 mm to (253.5, 98.7)
- moved SW2 131.4 mm to (186.7, 48.8), turned to 180 degrees
- moved SW51 106.9 mm to (39.2, 117.8)
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Connections:
- SW10 pad 1: (no net) -> unconnected-(SW10-Pad1)
- SW10 pad 2: (no net) -> Net-(D10-Pad2)
- SW11 pad 1: (no net) -> unconnected-(SW11-Pad1)
- SW11 pad 2: (no net) -> Net-(D11-Pad2)
- SW12 pad 1: (no net) -> unconnected-(SW12-Pad1)
- SW12 pad 2: (no net) -> Net-(D12-Pad2)
- SW13 pad 1: (no net) -> unconnected-(SW13-Pad1)
- SW13 pad 2: (no net) -> Net-(D13-Pad2)
- SW14 pad 1: (no net) -> unconnected-(SW14-Pad1)
- SW14 pad 2: (no net) -> Net-(D14-Pad2)
- SW15 pad 1: (no net) -> unconnected-(SW15-Pad1)
- SW15 pad 2: (no net) -> Net-(D15-Pad2)
- SW16 pad 1: (no net) -> unconnected-(SW16-Pad1)
- SW16 pad 2: (no net) -> Net-(D16-Pad2)
- SW17 pad 1: (no net) -> unconnected-(SW17-Pad1)
- SW17 pad 2: (no net) -> Net-(D17-Pad2)
- SW18 pad 1: (no net) -> unconnected-(SW18-Pad1)
- SW18 pad 2: (no net) -> Net-(D18-Pad2)
- SW19 pad 1: (no net) -> unconnected-(SW19-Pad1)
- SW19 pad 2: (no net) -> Net-(D19-Pad2)
- SW2 pad 1: (no net) -> unconnected-(SW2-Pad1)
- SW2 pad 2: (no net) -> GND
- SW20 pad 1: (no net) -> unconnected-(SW20-Pad1)
- SW20 pad 2: (no net) -> Net-(D20-Pad2)
- SW21 pad 1: (no net) -> unconnected-(SW21-Pad1)
- SW21 pad 2: (no net) -> Net-(D21-Pad2)
- SW22 pad 1: (no net) -> unconnected-(SW22-Pad1)
- SW22 pad 2: (no net) -> Net-(D22-Pad2)
- SW23 pad 1: (no net) -> unconnected-(SW23-Pad1)
- SW23 pad 2: (no net) -> Net-(D23-Pad2)
- SW24 pad 1: (no net) -> unconnected-(SW24-Pad1)
- SW24 pad 2: (no net) -> Net-(D24-Pad2)
- SW25 pad 1: (no net) -> unconnected-(SW25-Pad1)
- SW25 pad 2: (no net) -> Net-(D25-Pad2)
- SW26 pad 1: (no net) -> unconnected-(SW26-Pad1)
- SW26 pad 2: (no net) -> Net-(D26-Pad2)
- SW27 pad 1: (no net) -> unconnected-(SW27-Pad1)
- SW27 pad 2: (no net) -> Net-(D27-Pad2)
- SW29 pad 1: (no net) -> unconnected-(SW29-Pad1)
- SW29 pad 2: (no net) -> Net-(D29-Pad2)
- SW3 pad 1: (no net) -> unconnected-(SW3-Pad1)
- SW3 pad 2: (no net) -> Net-(D3-Pad2)
- SW30 pad 1: (no net) -> unconnected-(SW30-Pad1)
- SW30 pad 2: (no net) -> Net-(D30-Pad2)
- SW31 pad 1: (no net) -> unconnected-(SW31-Pad1)
- SW31 pad 2: (no net) -> Net-(D31-Pad2)
- SW32 pad 1: (no net) -> unconnected-(SW32-Pad1)
- SW32 pad 2: (no net) -> Net-(D32-Pad2)
- SW33 pad 1: (no net) -> unconnected-(SW33-Pad1)
- SW33 pad 2: (no net) -> Net-(D33-Pad2)
- SW34 pad 1: (no net) -> unconnected-(SW34-Pad1)
- SW34 pad 2: (no net) -> Net-(D34-Pad2)
- SW35 pad 1: (no net) -> unconnected-(SW35-Pad1)
- SW35 pad 2: (no net) -> Net-(D35-Pad2)
- SW36 pad 1: (no net) -> unconnected-(SW36-Pad1)
- SW36 pad 2: (no net) -> Net-(D36-Pad2)
- SW37 pad 1: (no net) -> unconnected-(SW37-Pad1)
- SW37 pad 2: (no net) -> Net-(D37-Pad2)
- SW38 pad 1: (no net) -> unconnected-(SW38-Pad1)
- SW38 pad 2: (no net) -> Net-(D38-Pad2)
- SW39 pad 1: (no net) -> unconnected-(SW39-Pad1)
- SW39 pad 2: (no net) -> Net-(D39-Pad2)
- SW4 pad 1: (no net) -> unconnected-(SW4-Pad1)
- SW4 pad 2: (no net) -> Net-(D4-Pad2)
- SW41 pad 1: (no net) -> unconnected-(SW41-Pad1)
- SW41 pad 2: (no net) -> Net-(D41-Pad2)
- SW42 pad 1: (no net) -> unconnected-(SW42-Pad1)
- SW42 pad 2: (no net) -> Net-(D42-Pad2)
- SW43 pad 1: (no net) -> unconnected-(SW43-Pad1)
- SW43 pad 2: (no net) -> Net-(D43-Pad2)
- SW44 pad 1: (no net) -> unconnected-(SW44-Pad1)
- SW44 pad 2: (no net) -> Net-(D44-Pad2)
- SW45 pad 1: (no net) -> unconnected-(SW45-Pad1)
- SW45 pad 2: (no net) -> Net-(D45-Pad2)
- SW46 pad 1: (no net) -> unconnected-(SW46-Pad1)
- SW46 pad 2: (no net) -> Net-(D46-Pad2)
- SW47 pad 1: (no net) -> unconnected-(SW47-Pad1)
- SW47 pad 2: (no net) -> Net-(D47-Pad2)
- SW48 pad 1: (no net) -> unconnected-(SW48-Pad1)
- SW48 pad 2: (no net) -> Net-(D48-Pad2)
- SW49 pad 1: (no net) -> unconnected-(SW49-Pad1)
- SW49 pad 2: (no net) -> Net-(D49-Pad2)
- SW5 pad 1: (no net) -> unconnected-(SW5-Pad1)
- SW5 pad 2: (no net) -> Net-(D5-Pad2)
- SW50 pad 1: (no net) -> unconnected-(SW50-Pad1)
- SW50 pad 2: (no net) -> Net-(D50-Pad2)
- SW51 pad 1: (no net) -> unconnected-(SW51-Pad1)
- SW51 pad 2: (no net) -> Net-(D51-Pad2)
- SW54 pad 1: (no net) -> unconnected-(SW54-Pad1)
- SW54 pad 2: (no net) -> Net-(D54-Pad2)
- SW55 pad 1: (no net) -> unconnected-(SW55-Pad1)
- SW55 pad 2: (no net) -> Net-(D55-Pad2)
- SW6 pad 1: (no net) -> unconnected-(SW6-Pad1)
- SW6 pad 2: (no net) -> Net-(D6-Pad2)
- SW7 pad 1: (no net) -> unconnected-(SW7-Pad1)
- SW7 pad 2: (no net) -> Net-(D7-Pad2)
- SW8 pad 1: (no net) -> unconnected-(SW8-Pad1)
- SW8 pad 2: (no net) -> Net-(D8-Pad2)
- SW9 pad 1: (no net) -> unconnected-(SW9-Pad1)
- SW9 pad 2: (no net) -> Net-(D9-Pad2)
Routing:
- net VBUS: track 0.00 -> 227.2 mm, vias 0 -> 3
- net D+: track 0.00 -> 199.6 mm
- net D-: track 0.00 -> 198.7 mm
- net DP+: track 0.00 -> 20.1 mm
- net DP-: track 0.00 -> 20.1 mm
- net Net-(J2-PadA5): track 0.00 -> 7.50 mm
- net GND: track 0.00 -> 5.66 mm, vias 0 -> 1
- net Net-(J2-PadB5): track 0.00 -> 2.84 mm
- net VDD: track 0.00 -> 0.65 mm
- added copper zone on B.Cu, net GND
- added copper zone on F.Cu, net GND
Other:
- board size 243.1 x 105 mm -> 238.1 x 106.4 mm

Commit message: Cập nhật Lmao
Parts:
- added C1: 10nF, Capacitor_SMD:C_0603_1608Metric_Pad1.08x0.95mm_HandSolder, F.Cu at (137.2, -7.62)
- added C10: C, Capacitor_SMD:C_0603_1608Metric_Pad1.08x0.95mm_HandSolder, F.Cu at (163.8, -7.28)
- added C11: C, Capacitor_SMD:C_0603_1608Metric_Pad1.08x0.95mm_HandSolder, F.Cu at (159.4, -7.28)
- added C12: C, Capacitor_SMD:C_0603_1608Metric_Pad1.08x0.95mm_HandSolder, F.Cu at (155.1, -7.28)
- added C13: C, Capacitor_SMD:C_0603_1608Metric_Pad1.08x0.95mm_HandSolder, F.Cu at (159.4, -14.8)
- added C14: C, Capacitor_SMD:C_0603_1608Metric_Pad1.08x0.95mm_HandSolder, F.Cu at (168.1, -17.3)
- added C15: C, Capacitor_SMD:C_0603_1608Metric_Pad1.08x0.95mm_HandSolder, F.Cu at (155.1, -17.3)
- added C16: C, Capacitor_SMD:C_0603_1608Metric_Pad1.08x0.95mm_HandSolder, F.Cu at (168.1, -9.79)
- added C17: C, Capacitor_SMD:C_0603_1608Metric_Pad1.08x0.95mm_HandSolder, F.Cu at (159.4, -17.3)
- added C18: C, Capacitor_SMD:C_0603_1608Metric_Pad1.08x0.95mm_HandSolder, F.Cu at (176.8, -17.3)
- added C19: C, Capacitor_SMD:C_0603_1608Metric_Pad1.08x0.95mm_HandSolder, F.Cu at (163.8, -9.79)
- added C2: 1nF, Capacitor_SMD:C_0603_1608Metric_Pad1.08x0.95mm_HandSolder, F.Cu at (136.1, -4.67)
- added C20: C, Capacitor_SMD:C_0603_1608Metric_Pad1.08x0.95mm_HandSolder, F.Cu at (163.8, -17.3)
- added C21: C, Capacitor_SMD:C_0603_1608Metric_Pad1.08x0.95mm_HandSolder, F.Cu at (163.8, -4.77)
- added C22: C, Capacitor_SMD:C_0603_1608Metric_Pad1.08x0.95mm_HandSolder, F.Cu at (168.1, -12.3)
- added C23: C, Capacitor_SMD:C_0603_1608Metric_Pad1.08x0.95mm_HandSolder, F.Cu at (159.4, -12.3)
- added C24: C, Capacitor_SMD:C_0603_1608Metric_Pad1.08x0.95mm_HandSolder, F.Cu at (176.8, -14.8)
- added C25: C, Capacitor_SMD:C_0603_1608Metric_Pad1.08x0.95mm_HandSolder, F.Cu at (168.1, -14.8)
- added C26: C, Capacitor_SMD:C_0603_1608Metric_Pad1.08x0.95mm_HandSolder, F.Cu at (155.1, -9.79)
- added C27: C, Capacitor_SMD:C_0603_1608Metric_Pad1.08x0.95mm_HandSolder, F.Cu at (163.8, -14.8)
- added C28: C, Capacitor_SMD:C_0603_1608Metric_Pad1.08x0.95mm_HandSolder, F.Cu at (155.1, -12.3)
- added C29: C, Capacitor_SMD:C_0603_1608Metric_Pad1.08x0.95mm_HandSolder, F.Cu at (155.1, -14.8)
- added C3: 10uF, Capacitor_Tantalum_SMD:CP_EIA-3216-12_Kemet-S_Pad1.58x1.35mm_HandSolder, F.Cu at (126.5, -5.90)
- added C30: C, Capacitor_SMD:C_0603_1608Metric_Pad1.08x0.95mm_HandSolder, F.Cu at (163.8, -12.3)
- added C31: C, Capacitor_SMD:C_0603_1608Metric_Pad1.08x0.95mm_HandSolder, F.Cu at (155.1, -4.77)
- added C32: C, Capacitor_SMD:C_0603_1608Metric_Pad1.08x0.95mm_HandSolder, F.Cu at (159.4, -9.79)
- added C33: C, Capacitor_SMD:C_0603_1608Metric_Pad1.08x0.95mm_HandSolder, F.Cu at (172.5, -14.8)
- added C34: C, Capacitor_SMD:C_0603_1608Metric_Pad1.08x0.95mm_HandSolder, F.Cu at (172.5, -12.3)
- added C35: C, Capacitor_SMD:C_0603_1608Metric_Pad1.08x0.95mm_HandSolder, F.Cu at (172.5, -17.3)
- added C4: 10uF, Capacitor_Tantalum_SMD:CP_EIA-3216-12_Kemet-S_Pad1.58x1.35mm_HandSolder, F.Cu at (133.0, -10.4)
- added C5: 10uF, Capacitor_SMD:C_0603_1608Metric_Pad1.08x0.95mm_HandSolder, F.Cu at (131.7, -4.67)
- added C9: C, Capacitor_SMD:C_0603_1608Metric_Pad1.08x0.95mm_HandSolder, F.Cu at (159.4, -4.77)
- added D1: BLUE, kien242:LED6028-3228-2pin, F.Cu at (121.9, 185.4)
- added D2: 1N5819, Diode_SMD:D_SOD-323_HandSoldering, F.Cu at (132.5, -7.40)
- added H10: Hole, MountingHole:MountingHole_2.5mm_Pad_Via, F.Cu at (113.7, -1.70)
- added H11: Hole, MountingHole:MountingHole_2.5mm_Pad_Via, F.Cu at (120.2, -8.25)
- added H12: Hole, MountingHole:MountingHole_2.5mm_Pad_Via, F.Cu at (120.2, -1.70)
- added H7: Hole, MountingHole:MountingHole_2.5mm_Pad_Via, F.Cu at (113.7, -8.25)
- added H8: Hole, MountingHole:MountingHole_2.5mm_Pad_Via, F.Cu at (129.8, -15.3)
- added H9: Hole, MountingHole:MountingHole_2.5mm_Pad_Via, F.Cu at (123.2, -15.3)
- added J1: , kien242:JST_PH_S2B-PH-SM4-TB_1x02-1MP_P2.00mm_Horizontal, F.Cu at (112.6, 188.9)
- added LED1: 6812, kien242:SK6812-MINI, F.Cu at (139.0, 165.0)
- added LED10: 6812, kien242:SK6812-MINI, F.Cu at (118.0, 160.0)
- added LED11: 6812, kien242:SK6812-MINI, F.Cu at (139.0, 160.0)
- added LED12: 6812, kien242:SK6812-MINI, F.Cu at (118.0, 165.0)
- added LED13: 6812, kien242:SK6812-MINI, F.Cu at (132.0, 165.0)
- added LED14: 6812, kien242:SK6812-MINI, F.Cu at (146.1, 154.9)
- added LED15: 6812, kien242:SK6812-MINI, F.Cu at (118.0, 170.1)
- added LED16: 6812, kien242:SK6812-MINI, F.Cu at (146.1, 160.0)
- added LED17: 6812, kien242:SK6812-MINI, F.Cu at (111.0, 160.0)
- added LED18: 6812, kien242:SK6812-MINI, F.Cu at (111.0, 170.1)
- added LED19: 6812, kien242:SK6812-MINI, F.Cu at (111.0, 165.0)
- added LED2: 6812, kien242:SK6812-MINI, F.Cu at (118.0, 154.9)
- added LED20: 6812, kien242:SK6812-MINI, F.Cu at (125.0, 160.0)
- added LED21: 6812, kien242:SK6812-MINI, F.Cu at (132.0, 175.1)
- added LED22: 6812, kien242:SK6812-MINI, F.Cu at (125.0, 175.1)
- added LED23: 6812, kien242:SK6812-MINI, F.Cu at (139.0, 154.9)
- added LED24: 6812, kien242:SK6812-MINI, F.Cu at (125.0, 154.9)
- added LED25: 6812, kien242:SK6812-MINI, F.Cu at (118.0, 175.1)
- added LED26: 6812, kien242:SK6812-MINI, F.Cu at (132.0, 160.0)
- added LED27: 6812, kien242:SK6812-MINI, F.Cu at (132.0, 154.9)
- added LED3: 6812, kien242:SK6812-MINI, F.Cu at (111.0, 154.9)
- added LED4: 6812, kien242:SK6812-MINI, F.Cu at (125.0, 165.0)
- added LED5: 6812, kien242:SK6812-MINI, F.Cu at (132.0, 170.1)
- added LED6: 6812, kien242:SK6812-MINI, F.Cu at (153.1, 154.9)
- added LED7: 6812, kien242:SK6812-MINI, F.Cu at (139.0, 170.1)
- added LED8: 6812, kien242:SK6812-MINI, F.Cu at (111.0, 175.1)
- added LED9: 6812, kien242:SK6812-MINI, F.Cu at (125.0, 170.1)
- added Q1: AO3407, Package_TO_SOT_SMD:SOT-23_Handsoldering, F.Cu at (126.7, -9.75)
- added Q2: AO3407, Package_TO_SOT_SMD:SOT-23_Handsoldering, F.Cu at (136.3, -16.3)
- added R1: 2m, Resistor_SMD:R_0603_1608Metric_Pad0.98x0.95mm_HandSolder, F.Cu at (131.5, -2.16)
- added R10: 100K, Resistor_SMD:R_0603_1608Metric_Pad0.98x0.95mm_HandSolder, F.Cu at (138.2, -10.2)
- added R3: 2m, Resistor_SMD:R_0603_1608Metric_Pad0.98x0.95mm_HandSolder, F.Cu at (142.5, -10.2)
- added R5: 2M, Resistor_SMD:R_0603_1608Metric_Pad0.98x0.95mm_HandSolder, F.Cu at (130.0, 1.58)
- added R6: 10M, Resistor_SMD:R_0603_1608Metric_Pad0.98x0.95mm_HandSolder, F.Cu at (125.7, 1.58)
- added R7: 1K, Resistor_SMD:R_0603_1608Metric_Pad0.98x0.95mm_HandSolder, F.Cu at (142.5, -12.7)
- added R8: RPROG, Resistor_SMD:R_0603_1608Metric_Pad0.98x0.95mm_HandSolder, F.Cu at (147.5, -17.3)
- added R9: 100K, Resistor_SMD:R_0603_1608Metric_Pad0.98x0.95mm_HandSolder, F.Cu at (138.2, -12.7)
- added SW1: SW_Push, Button_Switch_SMD:SW_SPST_TL3342, F.Cu at (115.2, -15.1)
- added U1: TP4054, Package_TO_SOT_SMD:SOT-23-5_HandSoldering, F.Cu at (142.4, -16.2)
- added U3: MIC5219-3.3YM5, Package_TO_SOT_SMD:SOT-23-5_HandSoldering, F.Cu at (126.4, -2.00)
- SW48: value 1u -> 1.25u; footprint MX-hotswap:SW-HS-1u -> MX-hotswap:SW-HS-1.25u
- SW50, SW60, SW62: value 1.25u -> 1u; footprint MX-hotswap:SW-HS-1.25u -> MX-hotswap:SW-HS-1u
- SW56: value 2u -> 2.75u; footprint MX-hotswap:SW-HS-2u -> MX-hotswap:SW-HS-2.75u
- SW57: value 1u -> 2u; footprint MX-hotswap:SW-HS-1u -> MX-hotswap:SW-HS-2u
- SW58: value 2.25u -> 1u; footprint MX-hotswap:SW-HS-2.25u -> MX-hotswap:SW-HS-1u
- moved SW57 23.8 mm to (170.2, 117.8)
- moved SW58 21.4 mm to (198.8, 117.8)
- moved SW60 7.14 mm to (217.8, 117.8)
- moved H2 7.14 mm to (124.9, 117.8), turned to 0 degrees
- moved SW56 7.14 mm to (124.9, 117.8)
- moved H3 7.14 mm to (170.2, 117.8), turned to 0 degrees
- moved SW49 4.76 mm to (236.9, 98.7)
- moved SW61 4.76 mm to (236.9, 117.8)
- moved SW48 2.38 mm to (215.4, 98.7)
- moved SW50 2.38 mm to (255.9, 98.7)
- moved SW62 2.38 mm to (255.9, 117.8)

Commit message: update
Parts:
- removed C33, C34, C35: C, Capacitor_SMD:C_0603_1608Metric_Pad1.08x0.95mm_HandSolder
- removed H10, H11, H12: Hole, MountingHole:MountingHole_2.5mm_Pad_Via
- removed the H7 at (113.7, -8.25)
- removed the J1 at (112.6, 188.9)
- removed the R1 at (131.5, -2.16)
- removed the U1 at (142.4, -16.2)
- added C6: C, Capacitor_SMD:C_0603_1608Metric_Pad1.08x0.95mm_HandSolder, B.Cu at (139.0, -42.9)
- added C7: C, Capacitor_SMD:C_0603_1608Metric_Pad1.08x0.95mm_HandSolder, B.Cu at (134.6, -45.4)
- added C8: C, Capacitor_SMD:C_0603_1608Metric_Pad1.08x0.95mm_HandSolder, B.Cu at (139.0, -45.4)
- added H2: Hole, MountingHole:MountingHole_2.5mm_Pad_Via, F.Cu at (92.7, -7.62)
- added H3: Hole, MountingHole:MountingHole_2.5mm_Pad_Via, F.Cu at (105.4, -15.2)
- added H5: Hole, MountingHole:MountingHole_2.5mm_Pad_Via, F.Cu at (99.1, -7.62)
- added H6: Hole, MountingHole:MountingHole_2.5mm_Pad_Via, F.Cu at (105.4, -7.62)
- added J3: , kien242:JST_PH_S2B-PH-SM4-TB_1x02-1MP_P2.00mm_Horizontal, B.Cu at (19.8, 1.78)
- added R4: 2m, Resistor_SMD:R_0603_1608Metric_Pad0.98x0.95mm_HandSolder, B.Cu at (31.1, -35.8)
- added U2: MS88FS3, kien242:MS88SF3-nRF52840, B.Cu at (102.1, 117.6)
- added U5: STM32F411CCUx, Package_DFN_QFN:QFN-48-1EP_7x7mm_P0.5mm_EP5.6x5.6mm, B.Cu at (102.1, 115.3)
- added kibuzzard-62F0EFF6: G***, kibuzzard-62F0EFF6, F.Cu at (102.1, 124.3)
- C1: value 10nF -> 10uF; moved to B.Cu
- C10, C11, C12, C13, C14, C15, C16, C17, C18, C19, C2, C20, C21, C22, C23, C24, C25, C26, C27, C28, C29, C30, C31, C32, C4, C9, D2, LED1, LED10, LED11, LED12, LED13, LED14, LED15, LED16, LED17, LED18, LED19, LED2, LED20, LED21, LED22, LED23, LED24, LED25, LED26, LED27, LED3, LED4, LED5, LED6, LED7, LED8, LED9, Q1, Q2, R10, R3, R7, SW1: moved to B.Cu
- C3: value 10uF -> 10nF; footprint Capacitor_Tantalum_SMD:CP_EIA-3216-12_Kemet-S_Pad1.58x1.35mm_HandSolder -> Capacitor_SMD:C_0603_1608Metric_Pad1.08x0.95mm_HandSolder; moved to B.Cu
- C5: footprint Capacitor_SMD:C_0603_1608Metric_Pad1.08x0.95mm_HandSolder -> Capacitor_Tantalum_SMD:CP_EIA-3216-12_Kemet-S_Pad1.58x1.35mm_HandSolder; moved to B.Cu
- R5: value 2M -> 10M; moved to B.Cu
- R6: value 10M -> 2M; moved to B.Cu
- R8: value RPROG -> 100K; moved to B.Cu
- R9: value 100K -> RPROG; moved to B.Cu
- U3: value MIC5219-3.3YM5 -> TP4054; moved to B.Cu
- U4: value MS88FS3 -> MIC5219-3.3YM5; footprint kien242:MS88SF3-nRF52840 -> Package_TO_SOT_SMD:SOT-23-5_HandSoldering
- moved LED21 232.0 mm to (154.9, -55.8), turned to 180 degrees
- moved LED18 231.5 mm to (161.9, -55.8), turned to 180 degrees
- moved LED7 230.1 mm to (182.9, -55.8), turned to 180 degrees
- moved LED22 228.9 mm to (161.9, -50.7), turned to 180 degrees
- moved LED8 228.3 mm to (168.9, -45.7), turned to 180 degrees
- moved LED4 221.7 mm to (175.9, -50.7), turned to 180 degrees
- moved LED17 218.5 mm to (168.9, -50.7), turned to 180 degrees
- moved LED25 218.5 mm to (175.9, -35.6), turned to 180 degrees
- moved LED3 218.5 mm to (168.9, -55.8), turned to 180 degrees
- moved LED5 217.8 mm to (161.9, -45.7), turned to 180 degrees
- moved LED10 215.7 mm to (182.9, -45.7), turned to 180 degrees
- moved LED23 213.9 mm to (175.9, -55.8), turned to 180 degrees
- moved LED15 210.9 mm to (182.9, -30.5), turned to 180 degrees
- moved U4 207.9 mm to (53.1, 1.27)
- moved LED6 207.8 mm to (182.9, -50.7), turned to 180 degrees
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- renumbered H2 to H4, H3 to H7, J2 to J1, R2 to R1, R4 to R2, SW41 to SW10, SW5 to SW11, SW17 to SW12, SW29 to SW13, SW54 to SW14, SW6 to SW15, SW18 to SW16, SW30 to SW17, SW42 to SW18, SW55 to SW19, SW7 to SW20, SW19 to SW21, SW31 to SW22, SW43 to SW23, SW8 to SW24, SW20 to SW25, SW32 to SW26, SW44 to SW27, SW56 to SW28, SW9 to SW29, SW21 to SW30, SW33 to SW31, SW45 to SW32, SW57 to SW33, SW10 to SW34, SW22 to SW35, SW34 to SW36, SW46 to SW37, SW58 to SW38, SW11 to SW39, SW15 to SW4, SW23 to SW40, SW35 to SW41, SW47 to SW42, SW12 to SW43, SW24 to SW44, SW36 to SW45, SW48 to SW46, SW60 to SW47, SW13 to SW48, SW25 to SW49, SW27 to SW5, SW37 to SW50, SW49 to SW51, SW61 to SW52, SW14 to SW53, SW26 to SW54, SW38 to SW55, SW50 to SW56, SW62 to SW57, SW39 to SW6, SW51 to SW7, SW4 to SW8, SW16 to SW9, U2 to U1
Connections:
- C1 pad 1: VBAT -> VDD
- C3 pad 1: Net-(C3-Pad1) -> VBAT
- C4 pad 1: VDD -> Net-(C4-Pad1)
- D2 pad 1: Net-(C3-Pad1) -> Net-(C4-Pad1)
- LED11 pad O: Net-(LED10-PadI) -> Net-(LED11-PadO)
- LED12 pad O: Net-(LED11-PadI) -> Net-(LED12-PadO)
- LED13 pad I: Net-(LED13-PadI) -> Net-(LED10-PadO)
- LED13 pad O: Net-(LED12-PadI) -> Net-(LED13-PadO)
- LED14 pad O: Net-(LED13-PadI) -> Net-(LED11-PadI)
- LED15 pad I: Net-(LED15-PadI) -> Net-(LED12-PadO)
- LED15 pad O: Net-(LED14-PadI) -> Net-(LED15-PadO)
- LED16 pad I: Net-(LED16-PadI) -> Net-(LED13-PadO)
- LED16 pad O: Net-(LED15-PadI) -> Net-(LED16-PadO)
- LED17 pad O: Net-(LED16-PadI) -> Net-(LED14-PadI)
- LED18 pad I: Net-(LED18-PadI) -> Net-(LED15-PadO)
- LED18 pad O: Net-(LED17-PadI) -> Net-(LED18-PadO)
- LED19 pad I: Net-(LED10-PadO) -> Net-(LED16-PadO)
- LED2 pad I: Net-(LED1-PadO) -> Net-(LED2-PadI)
- LED20 pad I: Net-(LED19-PadO) -> Net-(LED20-PadI)
- LED20 pad O: Net-(LED20-PadO) -> Net-(LED17-PadI)
- LED21 pad I: Net-(LED20-PadO) -> Net-(LED18-PadO)
- LED22 pad I: Net-(LED21-PadO) -> Net-(LED19-PadO)
- LED23 pad I: Net-(LED22-PadO) -> Net-(LED23-PadI)
- LED23 pad O: Net-(LED23-PadO) -> Net-(LED20-PadI)
- LED24 pad I: Net-(LED23-PadO) -> Net-(LED21-PadO)
- LED25 pad I: Net-(LED24-PadO) -> Net-(LED22-PadO)
- LED26 pad O: Net-(LED26-PadO) -> Net-(LED23-PadI)
- LED27 pad I: Net-(LED26-PadO) -> Net-(LED24-PadO)
- LED4 pad I: Net-(LED3-PadO) -> Net-(LED1-PadO)
- LED5 pad I: Net-(LED4-PadO) -> Net-(LED5-PadI)
- LED5 pad O: Net-(LED5-PadO) -> Net-(LED2-PadI)
- LED6 pad I: Net-(LED5-PadO) -> Net-(LED3-PadO)
- LED7 pad I: Net-(LED6-PadO) -> Net-(LED4-PadO)
- LED7 pad O: Net-(LED7-PadO) -> Net-(LED10-PadI)
- LED8 pad I: Net-(LED7-PadO) -> Net-(LED11-PadO)
- LED8 pad O: Net-(LED8-PadO) -> Net-(LED5-PadI)
- LED9 pad I: Net-(LED8-PadO) -> Net-(LED6-PadO)
- LED9 pad O: Net-(LED18-PadI) -> Net-(LED12-PadI)
- Q2 pad 2: Net-(C3-Pad1) -> Net-(C4-Pad1)
- R10 pad 1: VBUS -> Net-(C4-Pad1)
- R10 pad 2: GND -> BAT_CTR
- R3 pad 1: Net-(R1-Pad2) -> VBAT
- R3 pad 2: BATTERY_PIN -> Net-(R3-Pad2)
- R5 pad 1: POWER_PIN -> BATTERY_PIN
- R6 pad 1: BATTERY_PIN -> POWER_PIN
- R8 pad 1: Net-(R8-Pad1) -> VBUS
- R9 pad 1: Net-(C3-Pad1) -> Net-(R9-Pad1)
- R9 pad 2: BAT_CTR -> GND
- U3 pad 1: Net-(C3-Pad1) -> Net-(R7-Pad2)
- U3 pad 3: BAT_CTR -> VBAT
- U3 pad 4: unconnected-(U3-Pad4) -> VBUS
- U3 pad 5: VDD -> Net-(R9-Pad1)
- U4 pad 1: GND -> Net-(C4-Pad1)
- U4 pad 2: unconnected-(U4-Pad2) -> GND
- U4 pad 3: unconnected-(U4-Pad3) -> BAT_CTR
- U4 pad 5: ROW3 -> VDD
Routing:
- net VBUS: track 227.2 -> 24.7 mm
- net D+: track 199.6 -> 4.31 mm
- net D-: track 198.7 -> 4.72 mm
- net GND: track 5.66 -> 27.2 mm
- net DP-: track 20.1 -> 18.4 mm
- net DP+: track 20.1 -> 19.2 mm
- net VDD: track 0.65 -> 0.00 mm
