File: PCB/lmao/lmao.kicad_pcb (KiCad board)
At the start: 2 copper layers, 238.1 x 106.4 mm, 147 parts, among them J1 USB_C_Receptacle_USB2.0, J3 , Q1 AO3407, Q2 AO3407, SW1 SW_Push, SW10 1u, SW11 1u, SW12 1u, SW13 1u, SW14 1.25u, SW15 1u, SW16 1u, SW17 1u, SW18 1u, SW19 1.25u, SW2 , SW20 1u, SW21 1u, SW22 1u, SW23 1u, SW24 1u, SW25 1u, SW26 1u, SW27 1u, SW28 2.75u, SW29 1u, SW3 1u, SW30 1u, SW31 1u, SW32 1u, SW33 2u, SW34 1u, SW35 1u, SW36 1u, SW37 1u, SW38 1u, SW39 1u, SW4 1.5u, SW40 1u, SW41 1u, SW42 1u, SW43 1u, SW44 1u, SW45 1u, SW46 1.25u, SW47 1u, SW48 1u, SW49 1u, SW5 1.75u, SW50 1u, SW51 1u, SW52 1u, SW53 1u, SW54 1u, SW55 1.75u, SW56 1u, SW57 1u, SW6 2.25u, SW7 1.25u, SW8 1u, SW9 1u, U1 USBLC6-2SC6, U2 MS88FS3, U3 TP4054, U4 MIC5219-3.3YM5, U5 STM32F411CCUx

Commit message: update Lmao keyboard
Parts:
- removed the U2 at (102.1, 117.6)
- added JP1: , Jumper:SolderJumper-2_P1.3mm_Open_TrianglePad1.0x1.5mm, B.Cu at (31.0, -17.7)
- added JP2: , Jumper:SolderJumper-2_P1.3mm_Open_TrianglePad1.0x1.5mm, B.Cu at (52.3, 48.5)
- added LED28: , kien242:SK6812Mini-E, F.Cu at (255.9, 41.9)
- added LED29: , kien242:SK6812Mini-E, F.Cu at (236.9, 41.9)
- added LED30: , kien242:SK6812Mini-E, F.Cu at (217.8, 41.9)
- added LED31: , kien242:SK6812Mini-E, F.Cu at (198.8, 41.9)
- added LED32: , kien242:SK6812Mini-E, F.Cu at (174.9, 41.9)
- added LED33: , kien242:SK6812Mini-E, F.Cu at (155.9, 41.9)
- added LED34: , kien242:SK6812Mini-E, F.Cu at (136.8, 41.9)
- added LED35: , kien242:SK6812Mini-E, F.Cu at (117.8, 41.9)
- added LED36: , kien242:SK6812Mini-E, F.Cu at (94.0, 41.9)
- added LED37: , kien242:SK6812Mini-E, F.Cu at (74.9, 41.9)
- added LED38: , kien242:SK6812Mini-E, F.Cu at (55.9, 41.9)
- added LED39: , kien242:SK6812Mini-E, F.Cu at (36.8, 41.9)
- added LED40: , kien242:SK6812Mini-E, F.Cu at (41.6, 65.7)
- added LED41: , kien242:SK6812Mini-E, F.Cu at (65.4, 65.7)
- added LED42: , kien242:SK6812Mini-E, F.Cu at (84.5, 65.7)
- added LED43: , kien242:SK6812Mini-E, F.Cu at (103.5, 65.7)
- added LED44: , kien242:SK6812Mini-E, F.Cu at (122.6, 65.7)
- added LED45: , kien242:SK6812Mini-E, F.Cu at (141.6, 65.7)
- added LED46: , kien242:SK6812Mini-E, F.Cu at (160.7, 65.7)
- added LED47: , kien242:SK6812Mini-E, F.Cu at (179.7, 65.7)
- added LED48: , kien242:SK6812Mini-E, F.Cu at (198.8, 65.7)
- added LED49: , kien242:SK6812Mini-E, F.Cu at (217.8, 65.7)
- added LED50: , kien242:SK6812Mini-E, F.Cu at (236.9, 65.7)
- added LED51: , kien242:SK6812Mini-E, F.Cu at (255.9, 65.7)
- added LED52: , kien242:SK6812Mini-E, F.Cu at (248.8, 84.8)
- added LED53: , kien242:SK6812Mini-E, F.Cu at (222.6, 84.8)
- added LED54: , kien242:SK6812Mini-E, F.Cu at (203.5, 84.8)
- added LED55: , kien242:SK6812Mini-E, F.Cu at (184.5, 84.8)
- added LED56: , kien242:SK6812Mini-E, F.Cu at (165.4, 84.8)
- added LED57: , kien242:SK6812Mini-E, F.Cu at (146.4, 84.8)
- added LED58: , kien242:SK6812Mini-E, F.Cu at (127.3, 84.8)
- added LED59: , kien242:SK6812Mini-E, F.Cu at (108.3, 84.8)
- added LED60: , kien242:SK6812Mini-E, F.Cu at (89.2, 84.8)
- added LED61: , kien242:SK6812Mini-E, F.Cu at (70.2, 84.8)
- added LED62: , kien242:SK6812Mini-E, F.Cu at (44.0, 84.8)
- added LED63: , kien242:SK6812Mini-E, F.Cu at (48.7, 103.8)
- added LED64: , kien242:SK6812Mini-E, F.Cu at (79.7, 103.8)
- added LED65: , kien242:SK6812Mini-E, F.Cu at (98.7, 103.8)
- added LED66: , kien242:SK6812Mini-E, F.Cu at (117.8, 103.8)
- added LED67: , kien242:SK6812Mini-E, F.Cu at (136.8, 103.8)
- added LED68: , kien242:SK6812Mini-E, F.Cu at (155.9, 103.8)
- added LED69: , kien242:SK6812Mini-E, F.Cu at (174.9, 103.8)
- added LED70: , kien242:SK6812Mini-E, F.Cu at (194.0, 103.8)
- added LED71: , kien242:SK6812Mini-E, F.Cu at (215.4, 103.8)
- added LED72: , kien242:SK6812Mini-E, F.Cu at (236.9, 103.8)
- added LED73: , kien242:SK6812Mini-E, F.Cu at (255.9, 103.8)
- added LED74: , kien242:SK6812Mini-E, F.Cu at (255.9, 122.9)
- added LED75: , kien242:SK6812Mini-E, F.Cu at (236.9, 122.9)
- added LED76: , kien242:SK6812Mini-E, F.Cu at (217.8, 122.9)
- added LED77: , kien242:SK6812Mini-E, F.Cu at (198.8, 122.9)
- added LED78: , kien242:SK6812Mini-E, F.Cu at (170.2, 122.9)
- added LED79: , kien242:SK6812Mini-E, F.Cu at (124.9, 122.9)
- added LED80: , kien242:SK6812Mini-E, F.Cu at (86.8, 122.9)
- added LED81: , kien242:SK6812Mini-E, F.Cu at (63.0, 122.9)
- added LED82: , kien242:SK6812Mini-E, F.Cu at (39.2, 122.9)
- added SWD1: , kien242:SWD-4Pin, B.Cu at (113.0, 117.6)
- added U4: E73-2G4M08S1C, kien242:E73-2G4M08S1C, B.Cu at (102.4, 107.7)
- U5: value STM32F411CCUx -> STM32F401CBUx
- moved R9 66.1 mm to (57.7, 45.8), turned to 180 degrees
- moved C1 65.5 mm to (59.3, 48.9)
- moved J1 65.5 mm to (65.4, 48.9)
- moved U2 65.5 mm to (56.0, 48.5)
- moved SW1 64.9 mm to (45.8, 5.17), turned to 90 degrees
- moved R10 64.8 mm to (54.3, 45.8), turned to 0 degrees
- moved U5 45.5 mm to (147.6, 117.8)
- moved C15 13.3 mm to (130.3, -45.4)
- moved C21 13.3 mm to (130.3, -42.9)
- moved SW2 1.70 mm to (72.4, -21.6)
- moved R8 0.25 mm to (58.8, 8.26)
- moved Q2 0.25 mm to (59.8, 5.71)
- moved kibuzzard-62F0EFF6 0.25 mm to (102.4, 124.3)
- moved Q1 0.18 mm to (31.0, -20.8)
- moved R5 0.18 mm to (32.0, -23.4)
- renumbered C3 to C1, C4 to C3, C5 to C4, C1 to C5, D2 to D1, D1 to D2, H4 to H2, H7 to H3, H2 to H4, H8 to H6, H3 to H7, H6 to H8, J3 to J1, J1 to J2, LED2 to LED10, LED5 to LED11, LED8 to LED12, LED11 to LED13, LED17 to LED15, LED20 to LED16, LED23 to LED17, LED26 to LED18, LED3 to LED19, LED4 to LED2, LED6 to LED20, LED9 to LED21, LED12 to LED22, LED15 to LED23, LED18 to LED24, LED21 to LED25, LED24 to LED26, LED7 to LED3, LED10 to LED4, LED13 to LED5, LED16 to LED6, LED19 to LED7, LED22 to LED8, LED25 to LED9, R3 to R1, R9 to R10, R1 to R2, R4 to R3, R2 to R4, R6 to R5, R5 to R6, R10 to R7, R7 to R9, SW2 to SW1, SW34 to SW10, SW39 to SW11, SW43 to SW12, SW48 to SW13, SW53 to SW14, SW4 to SW15, SW9 to SW16, SW12 to SW17, SW16 to SW18, SW21 to SW19, SW1 to SW2, SW25 to SW20, SW30 to SW21, SW35 to SW22, SW40 to SW23, SW44 to SW24, SW49 to SW25, SW54 to SW26, SW5 to SW27, SW13 to SW28, SW17 to SW29, SW22 to SW30, SW26 to SW31, SW31 to SW32, SW36 to SW33, SW41 to SW34, SW45 to SW35, SW50 to SW36, SW55 to SW37, SW6 to SW38, SW10 to SW39, SW8 to SW4, SW18 to SW40, SW23 to SW41, SW27 to SW42, SW32 to SW43, SW37 to SW44, SW42 to SW45, SW51 to SW47, SW56 to SW48, SW7 to SW49, SW11 to SW5, SW14 to SW50, SW19 to SW51, SW28 to SW52, SW33 to SW53, SW38 to SW54, SW47 to SW55, SW52 to SW56, SW15 to SW6, SW20 to SW7, SW24 to SW8, SW29 to SW9, U4 to U1, U3 to U2, U1 to U3
Connections:
- D1 pad 2: VBUS -> +5V
- D2 pad 2: VBUS -> Net-(D2-Pad2)
- Q2 pad 1: VBUS -> +5V
- R8 pad 1: VBUS -> +5V
- U2 pad 4: VBUS -> Net-(D2-Pad2)
- U5 pad 23: unconnected-(U5-Pad23) -> GND1
- U5 pad 35: unconnected-(U5-Pad35) -> GND1
- U5 pad 47: unconnected-(U5-Pad47) -> GND1
- U5 pad 49: unconnected-(U5-Pad49) -> GND1
- U5 pad 8: unconnected-(U5-Pad8) -> GND1
Routing:
- net GND1: track 0.00 -> 21.3 mm, vias 0 -> 1
- net GND: track 27.2 -> 48.0 mm
- net Net-(C3-Pad1): track 0.00 -> 10.5 mm
- net VBUS: track 24.7 -> 30.6 mm
- net VBAT: track 0.00 -> 5.38 mm
- net SWDIO: track 0.00 -> 4.92 mm
- net SWCLK: track 0.00 -> 4.40 mm
- net +5V: track 0.00 -> 4.32 mm
- net Net-(R10-Pad1): track 0.00 -> 2.43 mm
- net Net-(D2-Pad2): track 0.00 -> 2.39 mm
- net VDD: track 0.00 -> 2.09 mm
- net Net-(R9-Pad2): track 0.00 -> 2.01 mm
- net BAT_CTR: track 0.00 -> 1.97 mm
- added copper zone on B.Cu, net GND1
- added copper zone on F.Cu, net GND1
