File: PCB/lmao/lmao.kicad_sch (KiCad schematic)
At the start: 37 parts, among them J1 , J2 USB_C_Receptacle_USB2.0, J4 SWD, Q1 AO3407, Q2 AO3407, SW1 SW_Push, SW2 , U1 TP4054, U2 USBLC6-2SC6, U3 MIC5219-3.3YM5, U4 MS88FS3

Commit message: update
Parts:
- added U5: STM32F411CCUx, Package_DFN_QFN:QFN-48-1EP_7x7mm_P0.5mm_EP5.6x5.6mm, symbol MCU_ST_STM32F4:STM32F411CCUx
- renumbered C5 to C1, C1 to C3, C3 to C4, C4 to C5, H7 to H2, H10 to H3, H2 to H4, H8 to H5, H11 to H6, H3 to H7, H9 to H8, H12 to H9, J2 to J1, J4 to J2, J1 to J3, R2 to R1, R9 to R10, R4 to R2, R1 to R3, R3 to R4, R6 to R5, R5 to R6, R10 to R8, R8 to R9, U2 to U1, U4 to U2, U1 to U3, U3 to U4
Connections:
- net GND: now also U2.63, U2.64

Commit message: update Lmao keyboard
Parts:
- removed J2: SWD, Library:SWD_Connector, symbol Connector_Generic:Conn_01x02
- removed U2: MS88FS3, kien242:MS88SF3-nRF52840, symbol kien242:MS88FS3
- removed U5: STM32F411CCUx, Package_DFN_QFN:QFN-48-1EP_7x7mm_P0.5mm_EP5.6x5.6mm, symbol MCU_ST_STM32F4:STM32F411CCUx
- added F1: 500mA, symbol Device:Polyfuse_Small
- added JP1, JP2: (no value), Jumper:SolderJumper-2_P1.3mm_Open_TrianglePad1.0x1.5mm, symbol Jumper:SolderJumper_2_Open
- added SWD1: (no value), kien242:SWD-4Pin, symbol kien242:SWD-STM32-4Pin
- added U4: E73-2G4M08S1C, kien242:E73-2G4M08S1C, symbol kien242:E73-2G4M08S1C
- renumbered C3 to C1, C4 to C3, C5 to C4, C1 to C5, D2 to D1, D1 to D2, H4 to H2, H7 to H3, H2 to H4, H8 to H6, H3 to H7, H6 to H8, J3 to J1, J1 to J2, R3 to R1, R9 to R10, R1 to R2, R4 to R3, R2 to R4, R6 to R5, R5 to R6, R10 to R7, R7 to R9, SW2 to SW1, SW1 to SW2, U4 to U1, U3 to U2, U1 to U3
Connections:
- net D+: now also U4.31 (D+)
- net D-: now also U4.29 (D-)
- net GND: now also SWD1.1 (GND), U4.21 (GND), U4.24 (GND), U4.5 (GND)
- net RST: now also U4.26 (P0.18/RESET)
- net SWCLK: now also SWD1.2 (CLK), U4.39 (SWDCLK)
- net SWDIO: now also SWD1.3 (DIO), U4.37 (SWDIO)
- net VBUS: now also F1.1, JP2.2 (B), U4.27 (VBUS); no longer D1.2 (A), D2.2 (A), Q2.1 (G), R8.1, U2.4 (VDD)
- net VCC: now also JP1.2 (B)
- net VDD: now also JP1.1 (A), SWD1.4 (3.3V), U4.19 (VDD), U4.23 (VDDH)
- new net: D2.2 (A), JP2.1 (A), U2.4 (VDD)
- new net +5V: D1.2 (A), F1.2, Q2.1 (G), R8.1
- no-connect marks 5 -> 2
Other:
- added sheet RGB_matrix (RGB_matrix.kicad_sch)
- added sheet STM32F401 (STM32F401.kicad_sch)
- moved on the sheet: C1, C3, C4, D1, D2, J1, Q2, R10, R7, R8, R9, SW1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
