File: PCB/lmao/matrix.kicad_sch (KiCad schematic)
At the start: 110 parts, among them SW10 1u, SW11 1u, SW12 1u, SW13 1u, SW14 1u, SW15 1.5u, SW16 1u, SW17 1u, SW18 1u, SW19 1u, SW20 1u, SW21 1u, SW22 1u, SW23 1u, SW24 1u, SW25 1u, SW26 1u, SW27 1.75u, SW29 1u, SW3 1u, SW30 1u, SW31 1u, SW32 1u, SW33 1u, SW34 1u, SW35 1u, SW36 1u, SW37 1u, SW38 1.75u, SW39 2.25u, SW4 1u, SW41 1u, SW42 1u, SW43 1u, SW44 1u, SW45 1u, SW46 1u, SW47 1u, SW48 1u, SW49 1u, SW5 1u, SW50 1.25u, SW51 1.25u, SW54 1.25u, SW55 1.25u, SW56 2u, SW57 1u, SW58 2.25u, SW6 1u, SW60 1.25u, SW61 1u, SW62 1.25u, SW7 1u, SW8 1u, SW9 1u

Commit message: Cập nhật Lmao
Parts:
- SW48: value 1u -> 1.25u; footprint MX-hotswap:SW-HS-1u -> MX-hotswap:SW-HS-1.25u
- SW50, SW60, SW62: value 1.25u -> 1u; footprint MX-hotswap:SW-HS-1.25u -> MX-hotswap:SW-HS-1u
- SW56: value 2u -> 2.75u; footprint MX-hotswap:SW-HS-2u -> MX-hotswap:SW-HS-2.75u
- SW57: value 1u -> 2u; footprint MX-hotswap:SW-HS-1u -> MX-hotswap:SW-HS-2u
- SW58: value 2.25u -> 1u; footprint MX-hotswap:SW-HS-2.25u -> MX-hotswap:SW-HS-1u
Changed lines of the file:
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@@
     (in_bom yes) (on_board yes) (fields_autoplaced)
     (property "Reference" "SW62" (id 0) (at 241.3 93.98 0))
-    (property "Value" "1.25u" (id 1) (at 241.3 96.52 0))
-    (property "Footprint" "MX-hotswap:SW-HS-1.25u" (id 2) (at 241.3 96.52 0)
+    (property "Value" "1u" (id 1) (at 241.3 96.52 0))
+    (property "Footprint" "MX-hotswap:SW-HS-1u" (id 2) (at 241.3 96.52 0)
       (effects (font (size 1.27 1.27)) hide)
     )
@@
     (in_bom yes) (on_board yes) (fields_autoplaced)
     (property "Reference" "SW50" (id 0) (at 241.3 74.93 0))
-    (property "Value" "1.25u" (id 1) (at 241.3 77.47 0))
-    (property "Footprint" "MX-hotswap:SW-HS-1.25u" (id 2) (at 241.3 77.47 0)
+    (property "Value" "1u" (id 1) (at 241.3 77.47 0))
+    (property "Footprint" "MX-hotswap:SW-HS-1u" (id 2) (at 241.3 77.47 0)
       (effects (font (size 1.27 1.27)) hide)
     )
@@
     (in_bom yes) (on_board yes) (fields_autoplaced)
     (property "Reference" "SW48" (id 0) (at 203.2 74.93 0))
-    (property "Value" "1u" (id 1) (at 203.2 77.47 0))
-    (property "Footprint" "MX-hotswap:SW-HS-1u" (id 2) (at 203.2 77.47 0)
+    (property "Value" "1.25u" (id 1) (at 203.2 77.47 0))
+    (property "Footprint" "MX-hotswap:SW-HS-1.25u" (id 2) (at 203.2 77.47 0)
       (effects (font (size 1.27 1.27)) hide)
     )
@@
     (in_bom yes) (on_board yes) (fields_autoplaced)
     (property "Reference" "SW57" (id 0) (at 146.05 93.98 0))
-    (property "Value" "1u" (id 1) (at 146.05 96.52 0))
-    (property "Footprint" "MX-hotswap:SW-HS-1u" (id 2) (at 146.05 96.52 0)
+    (property "Value" "2u" (id 1) (at 146.05 96.52 0))
+    (property "Footprint" "MX-hotswap:SW-HS-2u" (id 2) (at 146.05 96.52 0)
       (effects (font (size 1.27 1.27)) hide)
     )
@@
     (in_bom yes) (on_board yes) (fields_autoplaced)
     (property "Reference" "SW56" (id 0) (at 127 93.98 0))
-    (property "Value" "2u" (id 1) (at 127 96.52 0))
-    (property "Footprint" "MX-hotswap:SW-HS-2u" (id 2) (at 127 96.52 0)
+    (property "Value" "2.75u" (id 1) (at 127 96.52 0))
+    (property "Footprint" "MX-hotswap:SW-HS-2.75u" (id 2) (at 127 96.52 0)
       (effects (font (size 1.27 1.27)) hide)
     )
@@
     (in_bom yes) (on_board yes) (fields_autoplaced)
     (property "Reference" "SW58" (id 0) (at 165.1 93.98 0))
-    (property "Value" "2.25u" (id 1) (at 165.1 96.52 0))
-    (property "Footprint" "MX-hotswap:SW-HS-2.25u" (id 2) (at 165.1 96.52 0)
+    (property "Value" "1u" (id 1) (at 165.1 96.52 0))
+    (property "Footprint" "MX-hotswap:SW-HS-1u" (id 2) (at 165.1 96.52 0)
       (effects (font (size 1.27 1.27)) hide)
     )
@@
     (in_bom yes) (on_board yes) (fields_autoplaced)
     (property "Reference" "SW60" (id 0) (at 203.2 93.98 0))
-    (property "Value" "1.25u" (id 1) (at 203.2 96.52 0))
-    (property "Footprint" "MX-hotswap:SW-HS-1.25u" (id 2) (at 203.2 96.52 0)
-      (effects (font (size 1.27 1.27)) hide)
-    )
+    (property "Value" "1u" (id 1) (at 203.2 96.52 0))
+    (property "Footprint" "MX-hotswap:SW-HS-1u" (id 2) (at 203.2 96.52 0)
+      (effects (font (size 1.27 1.27)) hide)
+    )

Commit message: update
Parts:
- renumbered D41 to D10, D5 to D11, D17 to D12, D29 to D13, D54 to D14, D6 to D15, D18 to D16, D30 to D17, D42 to D18, D55 to D19, D7 to D20, D19 to D21, D31 to D22, D43 to D23, D8 to D24, D20 to D25, D32 to D26, D44 to D27, D56 to D28, D9 to D29, D21 to D30, D33 to D31, D45 to D32, D57 to D33, D10 to D34, D22 to D35, D34 to D36, D46 to D37, D58 to D38, D11 to D39, D15 to D4, D23 to D40, D35 to D41, D47 to D42, D12 to D43, D24 to D44, D36 to D45, D48 to D46, D60 to D47, D13 to D48, D25 to D49, D27 to D5, D37 to D50, D49 to D51, D61 to D52, D14 to D53, D26 to D54, D38 to D55, D50 to D56, D62 to D57, D39 to D6, D51 to D7, D4 to D8, D16 to D9, SW41 to SW10, SW5 to SW11, SW17 to SW12, SW29 to SW13, SW54 to SW14, SW6 to SW15, SW18 to SW16, SW30 to SW17, SW42 to SW18, SW55 to SW19, SW7 to SW20, SW19 to SW21, SW31 to SW22, SW43 to SW23, SW8 to SW24, SW20 to SW25, SW32 to SW26, SW44 to SW27, SW56 to SW28, SW9 to SW29, SW21 to SW30, SW33 to SW31, SW45 to SW32, SW57 to SW33, SW10 to SW34, SW22 to SW35, SW34 to SW36, SW46 to SW37, SW58 to SW38, SW11 to SW39, SW15 to SW4, SW23 to SW40, SW35 to SW41, SW47 to SW42, SW12 to SW43, SW24 to SW44, SW36 to SW45, SW48 to SW46, SW60 to SW47, SW13 to SW48, SW25 to SW49, SW27 to SW5, SW37 to SW50, SW49 to SW51, SW61 to SW52, SW14 to SW53, SW26 to SW54, SW38 to SW55, SW50 to SW56, SW62 to SW57, SW39 to SW6, SW51 to SW7, SW4 to SW8, SW16 to SW9

Commit message: update Lmao keyboard
Parts:
- renumbered D34 to D10, D39 to D11, D43 to D12, D48 to D13, D53 to D14, D4 to D15, D9 to D16, D12 to D17, D16 to D18, D21 to D19, D25 to D20, D30 to D21, D35 to D22, D40 to D23, D44 to D24, D49 to D25, D54 to D26, D5 to D27, D13 to D28, D17 to D29, D22 to D30, D26 to D31, D31 to D32, D36 to D33, D41 to D34, D45 to D35, D50 to D36, D55 to D37, D6 to D38, D10 to D39, D8 to D4, D18 to D40, D23 to D41, D27 to D42, D32 to D43, D37 to D44, D42 to D45, D51 to D47, D56 to D48, D7 to D49, D11 to D5, D14 to D50, D19 to D51, D28 to D52, D33 to D53, D38 to D54, D47 to D55, D52 to D56, D15 to D6, D20 to D7, D24 to D8, D29 to D9, SW34 to SW10, SW39 to SW11, SW43 to SW12, SW48 to SW13, SW53 to SW14, SW4 to SW15, SW9 to SW16, SW12 to SW17, SW16 to SW18, SW21 to SW19, SW25 to SW20, SW30 to SW21, SW35 to SW22, SW40 to SW23, SW44 to SW24, SW49 to SW25, SW54 to SW26, SW5 to SW27, SW13 to SW28, SW17 to SW29, SW22 to SW30, SW26 to SW31, SW31 to SW32, SW36 to SW33, SW41 to SW34, SW45 to SW35, SW50 to SW36, SW55 to SW37, SW6 to SW38, SW10 to SW39, SW8 to SW4, SW18 to SW40, SW23 to SW41, SW27 to SW42, SW32 to SW43, SW37 to SW44, SW42 to SW45, SW51 to SW47, SW56 to SW48, SW7 to SW49, SW11 to SW5, SW14 to SW50, SW19 to SW51, SW28 to SW52, SW33 to SW53, SW38 to SW54, SW47 to SW55, SW52 to SW56, SW15 to SW6, SW20 to SW7, SW24 to SW8, SW29 to SW9
