File: PCB/PCB/v1.1/MCU.kicad_sch (KiCad schematic)
At the start: 28 parts

Commit message: update file
Connections:
- net GND: now also U.21 (GND), U.24 (GND), U.5 (GND)
- net +3V3 renamed nRF_VDD
- net VCC renamed +3.3V
- no-connect marks 3 -> 4
Changed lines of the file:
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@@
-(kicad_sch (version 20220622) (generator eeschema)
+(kicad_sch (version 20220822) (generator eeschema)
   (paper "A4")
   (junction (at 118.745 42.545) (diameter 0) (color 0 0 0 0)
@@
   (junction (at 15.875 175.26) (diameter 0.9144) (color 0 0 0 0)
   )
-  (junction (at 144.145 42.545) (diameter 0) (color 0 0 0 0)
-  )
   (junction (at 42.545 43.18) (diameter 0) (color 0 0 0 0)
   )
   (junction (at 182.88 35.56) (diameter 0.9144) (color 0 0 0 0)
   )
+  (no_connect (at 146.05 139.7))
   (no_connect (at 42.545 54.61))
   (no_connect (at 133.985 45.085))
@@
     )
   )
-  (global_label "nRF_VDD" (shape input) (at 139.7 42.545 90) (fields_autoplaced)
+  (global_label "nRF_VDD" (shape input) (at 144.145 42.545 90) (fields_autoplaced)
     (effects (font (size 1.27 1.27)) (justify left))
-    (property "Intersheet References" "${INTERSHEET_REFS}" (id 0) (at 139.7794 32.117 90)
+    (property "Intersheet References" "${INTERSHEET_REFS}" (id 0) (at 144.2244 32.117 90)
       (effects (font (size 1.27 1.27)) (justify left) hide)
     )
@@
     )
   )
+  (global_label "nRF_VDD" (shape input) (at 230.505 43.18 270) (fields_autoplaced)
+    (effects (font (size 1.27 1.27)) (justify right))
+    (property "Intersheet References" "${INTERSHEET_REFS}" (id 0) (at 230.505 53.3766 90)
+      (effects (font (size 1.27 1.27)) (justify right) hide)
+    )
+  )
   (global_label "DP-" (shape input) (at 51.435 38.1 0) (fields_autoplaced)
     (effects (font (size 1.27 1.27)) (justify left))
@@
     )
     (property "Datasheet" "" (id 3) (at 126.365 52.705 0)
+      (effects (font (size 1.27 1.27)) hide)
+    )
+    (pin "1")
+  )
+  (symbol (lib_id "power:+3.3V") (at 230.505 24.13 0) (unit 1)
+    (in_bom yes) (on_board yes) (fields_autoplaced)
+    (default_instance (reference "#PWR?") (unit 1) (value "+3.3V") (footprint ""))
+    (property "Reference" "#PWR?" (id 0) (at 230.505 27.94 0)
+      (effects (font (size 1.27 1.27)) hide)
+    )
+    (property "Value" "+3.3V" (id 1) (at 230.505 20.32 0)
+      (effects (font (size 1.27 1.27)))
+    )
+    (property "Footprint" "" (id 2) (at 230.505 24.13 0)
+      (effects (font (size 1.27 1.27)) hide)
+    )
+    (property "Datasheet" "" (id 3) (at 230.505 24.13 0)
       (effects (font (size 1.27 1.27)) hide)
     )
@@
     (pin "S1")
   )
-  (symbol (lib_id "power:+3.3V") (at 144.145 42.545 0) (unit 1)
-    (in_bom yes) (on_board yes)
-    (default_instance (reference "U") (unit 1) (value "") (footprint ""))
-    (property "Reference" "U" (id 0) (at 144.145 46.355 0)
-      (effects (font (size 1.27 1.27)) hide)
-    )
-    (property "Value" "" (id 1) (at 144.145 36.83 0)
-      (effects (font (size 1.27 1.27)))
-    )
-    (property "Footprint" "" (id 2) (at 144.145 42.545 0)
-      (effects (font (size 1.27 1.27)) hide)
-    )
-    (property "Datasheet" "" (id 3) (at 144.145 42.545 0)
-      (effects (font (size 1.27 1.27)) hide)
-    )
-    (pin "1")
-  )
   (symbol (lib_id "Device:R_Small") (at 268.605 35.56 270) (unit 1)
     (in_bom yes) (on_board yes)
@@
     )
     (property "Datasheet" "" (id 3) (at 27.305 62.23 0)
+      (effects (font (size 1.27 1.27)) hide)
+    )
+    (pin "1")
+  )
+  (symbol (lib_id "power:GND") (at 135.89 139.7 0) (unit 1)
+    (in_bom yes) (on_board yes)
+    (default_instance (reference "#PWR?") (unit 1) (value "GND") (footprint ""))
+    (property "Reference" "#PWR?" (id 0) (at 135.89 146.05 0)
+      (effects (font (size 1.27 1.27)) hide)
+    )
+    (property "Value" "GND" (id 1) (at 135.89 146.05 90)
+      (effects (font (size 1.27 1.27)))
+    )
+    (property "Footprint" "" (id 2) (at 135.89 139.7 0)
+      (effects (font (size 1.27 1.27)) hide)
+    )
+    (property "Datasheet" "" (id 3) (at 135.89 139.7 0)
       (effects (font (size 1.27 1.27)) hide)
     )
@@
     (pin "2")
   )
+  (symbol (lib_id "power:GND") (at 143.51 137.16 0) (unit 1)
+    (in_bom yes) (on_board yes)
+    (default_instance (reference "#PWR?") (unit 1) (value "GND") (footprint ""))
+    (property "Reference" "#PWR?" (id 0) (at 143.51 143.51 0)
+      (effects (font (size 1.27 1.27)) hide)
+    )
+    (property "Value" "GND" (id 1) (at 143.51 143.51 90)
+      (effects (font (size 1.27 1.27)))
+    )
+    (property "Footprint" "" (id 2) (at 143.51 137.16 0)
+      (effects (font (size 1.27 1.27)) hide)
+    )
+    (property "Datasheet" "" (id 3) (at 143.51 137.16 0)
+      (effects (font (size 1.27 1.27)) hide)
+    )
+    (pin "1")
+  )
   (symbol (lib_id "Power_Protection:USBLC6-2SC6") (at 39.37 104.775 0) (mirror y) (unit 1)
     (in_bom yes) (on_board yes)
@@
     (pin "2")
   )
+  (symbol (lib_id "power:GND") (at 104.14 109.22 270) (unit 1)
+    (in_bom yes) (on_board yes)
+    (default_instance (reference "#PWR?") (unit 1) (value "GND") (footprint ""))
+    (property "Reference" "#PWR?" (id 0) (at 97.79 109.22 0)
+      (effects (font (size 1.27 1.27)) hide)
+    )
+    (property "Value" "GND" (id 1) (at 97.79 109.22 90)
+      (effects (font (size 1.27 1.27)))
+    )
+    (property "Footprint" "" (id 2) (at 104.14 109.22 0)
+      (effects (font (size 1.27 1.27)) hide)
+    )
+    (property "Datasheet" "" (id 3) (at 104.14 109.22 0)
+      (effects (font (size 1.27 1.27)) hide)
+    )
+    (pin "1")
+  )
   (symbol (lib_id "power:+5V") (at 15.875 175.26 0) (unit 1)
     (in_bom yes) (on_board yes) (fields_autoplaced)
@@
     (pin "1")
     (pin "2")
-  )
-  (symbol (lib_id "power:VCC") (at 230.505 24.13 0) (unit 1)
-    (in_bom yes) (on_board yes) (fields_autoplaced)
-    (default_instance (reference "U") (unit 1) (value "") (footprint ""))
-    (property "Reference" "U" (id 0) (at 230.505 27.94 0)
-      (effects (font (size 1.27 1.27)) hide)
-    )
-    (property "Value" "" (id 1) (at 230.505 18.415 0)
-      (effects (font (size 1.27 1.27)))
-    )
-    (property "Footprint" "" (id 2) (at 230.505 24.13 0)
-      (effects (font (size 1.27 1.27)) hide)
-    )
-    (property "Datasheet" "" (id 3) (at 230.505 24.13 0)
-      (effects (font (size 1.27 1.27)) hide)
-    )
-    (pin "1")
   )
   (symbol (lib_id "Device:C_Polarized_Small_US") (at 109.22 45.085 0) (unit 1)
@@
     (pin "2")
   )
-  (symbol (lib_id "power:+3.3V") (at 230.505 43.18 180) (unit 1)
-    (in_bom yes) (on_board yes) (fields_autoplaced)
-    (default_instance (reference "U") (unit 1) (value "") (footprint ""))
-    (property "Reference" "U" (id 0) (at 230.505 39.37 0)
-      (effects (font (size 1.27 1.27)) hide)
-    )
-    (property "Value" "" (id 1) (at 230.505 48.26 0)
-      (effects (font (size 1.27 1.27)))
-    )
-    (property "Footprint" "" (id 2) (at 230.505 43.18 0)
-      (effects (font (size 1.27 1.27)) hide)
-    )
-    (property "Datasheet" "" (id 3) (at 230.505 43.18 0)
-      (effects (font (size 1.27 1.27)) hide)
-    )
-    (pin "1")
-  )
   (symbol (lib_id "Device:C") (at 191.135 112.395 0) (unit 1)

Commit message: cap nhat PCB
Parts:
- added U: (no value), symbol Connector:USB_C_Receptacle_USB2.0
Connections:
- net +5V: now also U.A4 (VBUS), U.A9 (VBUS), U.B4 (VBUS), U.B9 (VBUS)
- net DP+: now also U.A6 (D+), U.B6 (D+)
- net DP-: now also U.A7 (D-), U.B7 (D-)
- net GND: now also U.A1 (GND), U.A12 (GND), U.B1 (GND), U.B12 (GND), U.S1 (SHIELD)
- net at U.1, U.A5 (CC1): now also U.B5 (CC2)
- net at U.2, U.B5 (CC2): now also U.A5 (CC1)
Changed lines of the file:
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@@
   (junction (at 126.365 52.705) (diameter 0) (color 0 0 0 0)
   )
+  (junction (at 42.545 24.13) (diameter 0) (color 0 0 0 0)
+  )
   (junction (at 42.545 38.1) (diameter 0) (color 0 0 0 0)
   )
   (junction (at 93.345 33.655) (diameter 0.9144) (color 0 0 0 0)
   )
+  (junction (at 42.545 39.37) (diameter 0) (color 0 0 0 0)
+  )
+  (junction (at 42.545 44.45) (diameter 0) (color 0 0 0 0)
+  )
   (junction (at 93.345 42.545) (diameter 0.9144) (color 0 0 0 0)
   )
   (junction (at 109.22 42.545) (diameter 0) (color 0 0 0 0)
   )
+  (junction (at 42.545 36.83) (diameter 0) (color 0 0 0 0)
+  )
+  (junction (at 42.545 41.91) (diameter 0) (color 0 0 0 0)
+  )
+  (junction (at 19.685 62.23) (diameter 0) (color 0 0 0 0)
+  )
   (junction (at 182.88 44.45) (diameter 0) (color 0 0 0 0)
   )
@@
   (junction (at 15.875 175.26) (diameter 0.9144) (color 0 0 0 0)
   )
+  (junction (at 42.545 31.75) (diameter 0) (color 0 0 0 0)
+  )
   (junction (at 42.545 43.18) (diameter 0) (color 0 0 0 0)
+  )
+  (junction (at 42.545 29.21) (diameter 0) (color 0 0 0 0)
   )
   (junction (at 182.88 35.56) (diameter 0.9144) (color 0 0 0 0)
@@
     (stroke (width 0) (type default))
   )
+  (wire (pts (xy 19.685 62.23) (xy 27.305 62.23))
+    (stroke (width 0) (type default))
+  )
   (wire (pts (xy 103.505 23.495) (xy 122.555 23.495))
     (stroke (width 0) (type default))
@@
   (wire (pts (xy 93.345 45.085) (xy 93.345 42.545))
     (stroke (width 0) (type solid))
-  )
-  (wire (pts (xy 19.685 62.23) (xy 27.305 62.23))
-    (stroke (width 0) (type default))
   )
   (text "RProg = 1000/IBat\nIBat in amps" (at 98.425 175.26 0)
@@
     (pin "1")
   )
+  (symbol (lib_name "USB_C_Receptacle_USB2.0_1") (lib_id "Connector:USB_C_Receptacle_USB2.0") (at 27.305 39.37 0) (unit 1)
+    (in_bom yes) (on_board yes) (fields_autoplaced)
+    (default_instance (reference "U") (unit 1) (value "") (footprint ""))
+    (property "Reference" "U" (id 0) (at 27.305 17.78 0)
+      (effects (font (size 1.27 1.27)))
+    )
+    (property "Value" "" (id 1) (at 27.305 20.32 0)
+      (effects (font (size 1.27 1.27)))
+    )
+    (property "Footprint" "" (id 2) (at 31.115 39.37 0)
+      (effects (font (size 1.27 1.27)) hide)
+    )
+    (property "Datasheet" "https://www.usb.org/sites/default/files/documents/usb_type-c.zip" (id 3) (at 31.115 39.37 0)
+      (effects (font (size 1.27 1.27)) hide)
+    )
+    (pin "A1")
+    (pin "A12")
+    (pin "A4")
+    (pin "A5")
+    (pin "A6")
+    (pin "A7")
+    (pin "A9")
+    (pin "B1")
+    (pin "B12")
+    (pin "B4")
+    (pin "B5")
+    (pin "B6")
+    (pin "B7")
+    (pin "B9")
+    (pin "S1")
+  )
   (symbol (lib_id "power:+5V") (at 93.345 33.655 0) (unit 1)
