File: PCB/PCB/v1.1/SofleKeyboard.kicad_sch (KiCad schematic)
At the start: 126 parts

Commit message: cap nhat PCB
Changed lines of the file:
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@@
     (pin "2")
   )
-  (sheet (at 95.25 165.1) (size 25.4 25.4) (fields_autoplaced)
+  (sheet (at 101.6 165.1) (size 25.4 25.4) (fields_autoplaced)
     (stroke (width 0.1524) (type solid))
     (fill (color 0 0 0 0.0000))
-    (property "Sheetname" "MCU" (id 0) (at 95.25 164.3884 0)
+    (property "Sheetname" "MCU" (id 0) (at 101.6 164.3884 0)
       (effects (font (size 1.27 1.27)) (justify left bottom))
     )
-    (property "Sheetfile" "MCU.kicad_sch" (id 1) (at 95.25 191.0846 0)
+    (property "Sheetfile" "MCU.kicad_sch" (id 1) (at 101.6 191.0846 0)
       (effects (font (size 1.27 1.27)) (justify left top))
     )
   )
-  (sheet (at 146.685 167.005) (size 25.4 25.4) (fields_autoplaced)
+  (sheet (at 139.7 165.1) (size 25.4 25.4) (fields_autoplaced)
     (stroke (width 0.1524) (type solid))
     (fill (color 0 0 0 0.0000))
-    (property "Sheetname" "RGB" (id 0) (at 146.685 166.2934 0)
+    (property "Sheetname" "RGB" (id 0) (at 139.7 164.3884 0)
       (effects (font (size 1.27 1.27)) (justify left bottom))
     )
-    (property "Sheetfile" "RGB.kicad_sch" (id 1) (at 146.685 192.9896 0)
+    (property "Sheetfile" "RGB.kicad_sch" (id 1) (at 139.7 191.0846 0)
       (effects (font (size 1.27 1.27)) (justify left top))
     )
@@
     )
     (path "/8eb96632-6a70-4ceb-bfd7-1fc7d35afecd/05f01b73-57ea-4049-affb-c6396c71a8b6"
-      (reference "J2") (unit 1) (value "USB_C_Receptacle_USB2.0") (footprint "kien242:USB-C-16pin-hight-v2")
+      (reference "J2") (unit 1) (value " ") (footprint "kien242:USB-C-16pin-hight-v2")
     )
     (path "/aad6a9d4-803c-48a9-8c48-ac14196e300b"
@@
       (reference "J4") (unit 1) (value " ") (footprint "Connector_JST:JST_PH_S2B-PH-K_1x02_P2.00mm_Horizontal")
     )
+    (path "/8eb96632-6a70-4ceb-bfd7-1fc7d35afecd/eda234e2-5758-44a6-964d-f2425118c536"
+      (reference "J5") (unit 1) (value " ") (footprint "kien242:USB-C-16pin-hight-v2")
+    )
     (path "/861bc896-4f06-45d4-8846-f0f9cb70383c"
